File: pcb/BMS.sch (KiCad schematic (older format))
At the start: 26 parts, among them Q1 PZT3906, SW2 SW_SPDT, U4 MCP73833, U5 LM8364-2.2, U6 LTC3525-5

Commit message: Most pcb of layout done
Parts:
- SW2: footprint SVastaCustomParts:E-Switch_Toggle_100SP1T1B4M2QE -> SVastaCustomParts:400BWMSP1R2BLKSM6QE‎_rocker_switch
Changed lines of the file:
@@
 F 0 "SW2" H 4800 1385 50  0000 C CNN
 F 1 "SW_SPDT" H 4800 1294 50  0000 C CNN
-F 2 "SVastaCustomParts:E-Switch_Toggle_100SP1T1B4M2QE" H 4800 1100 50  0001 C CNN
-F 3 "https://www.digikey.com/product-detail/en/100SP1T1B4M2QE/EG2355-ND/378824/?itemSeq=306854737" H 4800 1100 50  0001 C CNN
+F 2 "SVastaCustomParts:400BWMSP1R2BLKSM6QE‎_rocker_switch" H 4800 1100 50  0001 C CNN
+F 3 "https://www.digikey.com/product-detail/en/400BWMSP1R2BLKSM6QE/EG4336CT-ND/668634/?itemSeq=322026415" H 4800 1100 50  0001 C CNN
 	1    4800 1100
 	1    0    0    -1

Commit message: More layout work
Parts:
- D101, D102: footprint Keyboard_Parts:D_axial -> SVastaCustomParts:D_MiniMELF_Handsoldering_Shorter_Pads
Changed lines of the file:
@@
 F 0 "D102" V 3304 2029 50  0000 L CNN
 F 1 "D" V 3395 2029 50  0000 L CNN
-F 2 "Keyboard_Parts:D_axial" H 3350 1950 50  0001 C CNN
+F 2 "SVastaCustomParts:D_MiniMELF_Handsoldering_Shorter_Pads" H 3350 1950 50  0001 C CNN
 F 3 "~" H 3350 1950 50  0001 C CNN
 	1    3350 1950
@@
 F 0 "D101" H 3700 1316 50  0000 C CNN
 F 1 "D" H 3700 1225 50  0000 C CNN
-F 2 "Keyboard_Parts:D_axial" H 3700 1100 50  0001 C CNN
+F 2 "SVastaCustomParts:D_MiniMELF_Handsoldering_Shorter_Pads" H 3700 1100 50  0001 C CNN
 F 3 "~" H 3700 1100 50  0001 C CNN
 	1    3700 1100
