File: pcb/Keeb.kicad_pcb (KiCad board)
At the start: 2 copper layers, 340.4 x 121.9 mm, 177 parts, among them J1 TRRS_SJ1-42514, K00 KEYSW, K01 KEYSW, K02 KEYSW, K03 KEYSW, K04 KEYSW, K05 KEYSW, K10 KEYSW, K11 KEYSW, K12 KEYSW, K13 KEYSW, K14 KEYSW, K15 KEYSW, K20 KEYSW, K21 KEYSW, K22 KEYSW, K23 KEYSW, K24 KEYSW, K25 KEYSW, K26 KEYSW, K27 KEYSW, K30 KEYSW, K31 KEYSW, K32 KEYSW, K33 KEYSW, K34 KEYSW, K35 KEYSW, K36 KEYSW, K37 KEYSW, K42 KEYSW, K43 KEYSW, K44 KEYSW, K45 KEYSW, K46 KEYSW, K47 KEYSW, K52 KEYSW, K53 KEYSW, K54 KEYSW, K55 KEYSW, K56 KEYSW, K57 KEYSW, K60 KEYSW, K61 KEYSW, K62 KEYSW, K63 KEYSW, K64 KEYSW, K65 KEYSW, K66 KEYSW, K67 KEYSW, K70 KEYSW, K71 KEYSW, K72 KEYSW, K73 KEYSW, K74 KEYSW, K75 KEYSW, K76 KEYSW, K77 KEYSW, Q1 PZT3906, SW1 SW_RST, SW2 SW_SPDT, U1 ATMEGA32U4, U2 SN74HC138D‎, U3 SN74HC251, U4 MCP73833, U5 LM8364-2.2, U6 LTC3525-5, X1 XTAL_GND

Commit message: Layout & cad work for split pcb design
Parts:
- removed the D504 at (430.3, 248.8)
- added D500: D, SVastaCustomParts:D_MiniMELF_Handsoldering_Shorter_Pads, F.Cu at (411.8, 248.8)
- added REF**: PinHeader_1x12_P2.54mm_Vertical, Connector_PinHeader_2.54mm:PinHeader_1x12_P2.54mm_Vertical, F.Cu at (405.0, 217.6)
- added REF**: PinHeader_1x12_P2.54mm_Vertical, Connector_PinHeader_2.54mm:PinHeader_1x12_P2.54mm_Vertical, F.Cu at (438.1, 217.6)
- moved D302 52.8 mm to (436.2, 200.0)
- moved R18 52.8 mm to (431.3, 200.0)
- moved R7 39.7 mm to (411.8, 214.7), turned to 0 degrees
- moved R19 38.2 mm to (436.2, 211.7)
- moved R12 36.6 mm to (428.4, 187.4)
- moved D402 34.1 mm to (436.2, 203.9), turned to 180 degrees
- moved D401 33.1 mm to (436.2, 207.8), turned to 180 degrees
- moved D202 29.3 mm to (433.2, 191.3)
- moved D203 28.3 mm to (433.2, 195.2)
- moved R11 28.3 mm to (428.4, 191.3)
- moved D501 22.8 mm to (411.8, 252.7), turned to 0 degrees
- moved D503 22.5 mm to (411.8, 260.5), turned to 0 degrees
- moved D506 22.5 mm to (431.3, 256.6), turned to 0 degrees
- moved D504 22.4 mm to (431.3, 248.8), turned to 0 degrees
- moved JP1 20.7 mm to (404.0, 190.3), turned to 270 degrees
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- renumbered D505 to D501, D506 to D502, D507 to D503, D500 to D504, D501 to D505, D502 to D506, D503 to D507
Connections:
- D302 pad 2: Net-(D302-Pad2) -> /BatLow
- D501 pad 1: /SwitchMatrix/Col5 -> /SwitchMatrix/Col1
- D502 pad 1: /SwitchMatrix/Col6 -> /SwitchMatrix/Col2
- D503 pad 1: /SwitchMatrix/Col7 -> /SwitchMatrix/Col3
- D504 pad 1: /SwitchMatrix/Col0 -> /SwitchMatrix/Col4
- D505 pad 1: /SwitchMatrix/Col1 -> /SwitchMatrix/Col5
- D506 pad 1: /SwitchMatrix/Col2 -> /SwitchMatrix/Col6
- D507 pad 1: /SwitchMatrix/Col3 -> /SwitchMatrix/Col7
- U1 pad 20: Net-(D302-Pad2) -> Net-(U1-Pad20)
- U1 pad 25: Net-(U1-Pad25) -> RowSelectA
- U1 pad 26: Net-(U1-Pad26) -> RowSelectB
- U1 pad 27: /CapsLock -> RowSelectC
- U1 pad 28: /NumLock -> RowEnable
- U1 pad 29: RowSelectA -> ColSelectC
- U1 pad 30: /VbatMonitor -> ColSelectB
- U1 pad 31: RowSelectB -> ColEnable
- U1 pad 32: RowSelectC -> ColSelectA
- U1 pad 36: RowEnable -> ColValue
- U1 pad 37: ColSelectC -> /CapsLock
- U1 pad 38: ColSelectB -> /NumLock
- U1 pad 39: ColEnable -> /VbatMonitor
- U1 pad 40: ColSelectA -> /BatLow
- U1 pad 41: ColValue -> Net-(U1-Pad41)
- U3 pad 1: /SwitchMatrix/Col3 -> /SwitchMatrix/Col7
- U3 pad 12: /SwitchMatrix/Col7 -> /SwitchMatrix/Col3
- U3 pad 13: /SwitchMatrix/Col6 -> /SwitchMatrix/Col2
- U3 pad 14: /SwitchMatrix/Col5 -> /SwitchMatrix/Col1
- U3 pad 15: /SwitchMatrix/Col4 -> /SwitchMatrix/Col0
- U3 pad 2: /SwitchMatrix/Col2 -> /SwitchMatrix/Col6
- U3 pad 3: /SwitchMatrix/Col1 -> /SwitchMatrix/Col5
- U3 pad 4: /SwitchMatrix/Col0 -> /SwitchMatrix/Col4
Routing:
- net VCC: track 263.5 -> 197.1 mm
- net Net-(D302-Pad2): track 45.4 -> 0.00 mm
- net Net-(D500-Pad2): track 0.00 -> 45.2 mm, vias 0 -> 2
- net SCK: track 55.4 -> 13.3 mm, vias 1 -> 0
- net MISO: track 52.3 -> 10.8 mm, vias 1 -> 0
- net MOSI: track 53.6 -> 12.6 mm, vias 1 -> 0
- net SS1: track 55.3 -> 15.1 mm, vias 1 -> 0
- net /VbatMonitor: track 72.7 -> 33.8 mm, vias 2 -> 0
- net /SwitchMatrix/Col3: track 152.8 -> 184.7 mm, vias 0 -> 2
- net /SwitchMatrix/Col0: track 277.5 -> 308.4 mm, vias 0 -> 2
- net /IRQ: track 50.8 -> 20.8 mm, vias 1 -> 2
- net /SwitchMatrix/Col1: track 193.7 -> 223.5 mm, vias 0 -> 2
- net /SwitchMatrix/Col2: track 170.1 -> 199.0 mm, vias 0 -> 2
- net /RST: track 69.3 -> 42.8 mm
- net SCL: track 38.8 -> 56.1 mm
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Other:
- board text added: "Bat. Low"
- board text added: "Caps"
- board text added: "Num"
- board text removed: "Bat Low"
- board text removed: "CAPS"
- board text removed: "NUM"
