File: pcb/Keeb.kicad_pcb (KiCad board)
At the start: 2 copper layers, 343 x 150.5 mm, 178 parts, among them J1 TRRS_SJ1-42514, J2 TRRS_SJ1-42514, K0 KEYSW, K1 KEYSW, K10 KEYSW, K11 KEYSW, K12 KEYSW, K13 KEYSW, K14 KEYSW, K15 KEYSW, K2 KEYSW, K20 KEYSW, K21 KEYSW, K22 KEYSW, K23 KEYSW, K24 KEYSW, K25 KEYSW, K26 KEYSW, K27 KEYSW, K3 KEYSW, K30 KEYSW, K31 KEYSW, K32 KEYSW, K33 KEYSW, K34 KEYSW, K35 KEYSW, K36 KEYSW, K37 KEYSW, K4 KEYSW, K42 KEYSW, K43 KEYSW, K44 KEYSW, K45 KEYSW, K46 KEYSW, K47 KEYSW, K5 KEYSW, K52 KEYSW, K53 KEYSW, K54 KEYSW, K55 KEYSW, K56 KEYSW, K57 KEYSW, K60 KEYSW, K61 KEYSW, K62 KEYSW, K63 KEYSW, K64 KEYSW, K65 KEYSW, K66 KEYSW, K67 KEYSW, K70 KEYSW, K71 KEYSW, K72 KEYSW, K73 KEYSW, K74 KEYSW, K75 KEYSW, K76 KEYSW, K77 KEYSW, Q1 PZT3906, SW1 SW_RST, SW2 SW_SPDT, U1 ATMEGA32U4, U2 CD74AC138E, U3 CD74AC151E, U4 MCP73833, U5 LM8364-2.2, U6 LTC3525-5, X1 XTAL_GND

Commit message: Fixed some mistakes in logic/layout from v1
Parts:
- removed J2: TRRS_SJ1-42514, SVastaCustomParts:3.5mm_Cut_out
- D500, D501, D502, D503, D504, D505, D506, D507: footprint Keyboard_Parts:D_axial -> Diode_SMD:D_0805_2012Metric_Pad1.15x1.40mm_HandSolder
- R20: footprint Resistor_SMD:R_0805_2012Metric_Pad1.15x1.40mm_HandSolder -> Resistor_THT:R_Axial_DIN0204_L3.6mm_D1.6mm_P5.08mm_Horizontal
- moved D401 104.8 mm to (403.7, 117.6), turned to 90 degrees
- moved D402 104.4 mm to (406.3, 117.6), turned to 90 degrees
- moved R19 103.8 mm to (405.0, 121.4)
- moved D500 15.7 mm to (410.7, 167.8)
- moved R8 15.3 mm to (346.6, 74.4), turned to 0 degrees
- moved R20 14.8 mm to (417.1, 142.4), turned to 180 degrees
- moved R7 13.5 mm to (346.6, 77.0), turned to 0 degrees
- moved D507 13.3 mm to (418.3, 146.2)
- moved J1 12.7 mm to (343.4, 63.6)
- moved D501 12.0 mm to (410.7, 160.2)
- moved D506 10.9 mm to (418.3, 152.5)
- moved D502 8.52 mm to (410.7, 152.5)
- moved D505 7.41 mm to (418.3, 160.2)
- moved D503 6.35 mm to (410.7, 146.2)
- moved D504 4.58 mm to (418.3, 167.8)
Connections:
- J1 pad 2: SDA -> SCL
- J1 pad 3: SCL -> SDA
- U1 pad 21: /CapsLock -> Net-(U1-Pad21)
- U1 pad 22: /NumLock -> Net-(U1-Pad22)
- U1 pad 27: Net-(U1-Pad27) -> /CapsLock
- U1 pad 28: Net-(U1-Pad28) -> /NumLock
Routing:
- net /CapsLock: track 113.4 -> 11.2 mm
- net /NumLock: track 108.8 -> 9.82 mm
- net SCL: track 127.1 -> 84.5 mm, vias 3 -> 0
- net VCC: track 334.5 -> 308.1 mm
- net SDA: track 112.5 -> 93.6 mm, vias 2 -> 0
- net Net-(D500-Pad2): track 37.2 -> 52.6 mm, vias 0 -> 2
- net /SwitchMatrix/Row0: track 70.6 -> 85.5 mm
- net /SwitchMatrix/Row7: track 69.9 -> 56.8 mm
- net /SwitchMatrix/Row1: track 56.9 -> 68.0 mm
- net /SwitchMatrix/Row6: track 67.5 -> 56.9 mm
- net Net-(D401-Pad1): track 8.11 -> 0.00 mm
- net /SwitchMatrix/Row2: track 55.1 -> 62.3 mm
- net GND: track 86.7 -> 79.4 mm, vias 34 -> 31
- net /SwitchMatrix/Row5: track 74.4 -> 67.6 mm
- net /SwitchMatrix/Row3: track 58.0 -> 62.7 mm
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Other:
- outline, holes or cut-outs redrawn
- board text added: "C"
- board text added: "N"
- board text removed: "CAPS"
- board text removed: "NUM"

Commit message: Most pcb of layout done
Parts:
- removed D0, D1, D2, D3, D4, D5: D, Keyboard_Parts:D_axial
- removed K0, K1, K2, K3, K4, K5: KEYSW, keyswitches:Kailh_socket_vias
- added D00: D, Diode_SMD:D_1806_4516Metric_Pad1.57x1.80mm_HandSolder, F.Cu at (313.3, 126.9)
- added D01: D, Diode_SMD:D_1806_4516Metric_Pad1.57x1.80mm_HandSolder, F.Cu at (319.2, 126.9)
- added D02: D, Diode_SMD:D_1806_4516Metric_Pad1.57x1.80mm_HandSolder, F.Cu at (325.0, 126.9)
- added D03: D, Diode_SMD:D_1806_4516Metric_Pad1.57x1.80mm_HandSolder, F.Cu at (330.9, 126.9)
- added D04: D, Diode_SMD:D_1806_4516Metric_Pad1.57x1.80mm_HandSolder, F.Cu at (336.7, 126.9)
- added D05: D, Diode_SMD:D_1806_4516Metric_Pad1.57x1.80mm_HandSolder, F.Cu at (342.6, 126.9)
- added K00: KEYSW, keyswitches:Kailh_socket_via_on_pin_one, F.Cu at (275.4, 153.8)
- added K01: KEYSW, keyswitches:Kailh_socket_via_on_pin_one, F.Cu at (294.5, 157.9)
- added K02: KEYSW, keyswitches:Kailh_socket_via_on_pin_one, F.Cu at (314.3, 158.5)
- added K03: KEYSW, keyswitches:Kailh_socket_via_on_pin_one, F.Cu at (334.1, 159.1)
- added K04: KEYSW, keyswitches:Kailh_socket_via_on_pin_one, F.Cu at (352.5, 166.6)
- added K05: KEYSW, keyswitches:Kailh_socket_via_on_pin_one, F.Cu at (371.5, 170.7)
- D10, D11, D12, D13, D14, D15, D20, D21, D22, D23, D24, D25, D26, D27, D30, D31, D32, D33, D34, D35, D36, D37, D42, D43, D44, D45, D46, D47, D52, D53, D54, D55, D56, D57, D60, D61, D62, D63, D64, D65, D66, D67, D70, D71, D72, D73, D74, D75, D76, D77: footprint Keyboard_Parts:D_axial -> Diode_SMD:D_1806_4516Metric_Pad1.57x1.80mm_HandSolder
- JP1: moved to F.Cu
- K10, K11, K12, K13, K14, K15, K20, K21, K22, K23, K24, K25, K26, K27, K30, K31, K32, K33, K34, K35, K36, K37, K42, K43, K44, K45, K46, K47, K52, K53, K54, K55, K56, K57, K60, K61, K62, K63, K64, K65, K66, K67, K70, K71, K72, K73, K74, K75, K76, K77: footprint keyswitches:Kailh_socket_vias -> keyswitches:Kailh_socket_via_on_pin_one
- R3, R4, USB1: moved to B.Cu
- SW2: footprint SVastaCustomParts:E-Switch_Toggle_100SP1T1B4M2QE -> SVastaCustomParts:400BWMSP1R2BLKSM6QE‎_rocker_switch; moved to B.Cu
- U2: value CD74AC138E -> SN74HC138D‎; footprint SVastaCustomParts:CD74AC151_DIP-16 -> SVastaCustomParts:SN74HC_package_d_soic
- U3: value CD74AC151E -> SN74HC251; footprint SVastaCustomParts:CD74AC151_DIP-16 -> SVastaCustomParts:SN74HC_package_d_soic
- moved D77 154.6 mm to (548.2, 251.5)
- moved D67 154.4 mm to (545.8, 240.0)
- moved D76 152.6 mm to (542.5, 252.7)
- moved D66 152.3 mm to (540.1, 241.3)
- moved D30 151.0 mm to (284.1, 249.5)
- moved D20 150.8 mm to (286.6, 238.1)
- moved D75 150.5 mm to (536.8, 253.9)
- moved D65 150.3 mm to (534.3, 242.5)
- moved D36 149.6 mm to (380.6, 291.7), turned to 90 degrees
- moved D26 149.4 mm to (380.6, 280.0), turned to 90 degrees
- moved D31 149.0 mm to (289.9, 250.7)
- moved D21 148.8 mm to (292.3, 239.3)
- moved D74 148.5 mm to (531.0, 255.1)
- moved D64 148.3 mm to (528.6, 243.7)
- moved D37 147.3 mm to (386.4, 291.7), turned to 90 degrees
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Connections:
- net RowValue renamed ColValue
- D10 pad 1: /SwitchMatrix/Row1 -> /SwitchMatrix/Col0
- D11 pad 1: /SwitchMatrix/Row1 -> /SwitchMatrix/Col1
- D12 pad 1: /SwitchMatrix/Row1 -> /SwitchMatrix/Col2
- D13 pad 1: /SwitchMatrix/Row1 -> /SwitchMatrix/Col3
- D14 pad 1: /SwitchMatrix/Row1 -> /SwitchMatrix/Col4
- D15 pad 1: /SwitchMatrix/Row1 -> /SwitchMatrix/Col5
- D20 pad 1: /SwitchMatrix/Row2 -> /SwitchMatrix/Col0
- D21 pad 1: /SwitchMatrix/Row2 -> /SwitchMatrix/Col1
- D22 pad 1: /SwitchMatrix/Row2 -> /SwitchMatrix/Col2
- D23 pad 1: /SwitchMatrix/Row2 -> /SwitchMatrix/Col3
- D24 pad 1: /SwitchMatrix/Row2 -> /SwitchMatrix/Col4
- D25 pad 1: /SwitchMatrix/Row2 -> /SwitchMatrix/Col5
- D26 pad 1: /SwitchMatrix/Row2 -> /SwitchMatrix/Col6
- D27 pad 1: /SwitchMatrix/Row2 -> /SwitchMatrix/Col7
- D30 pad 1: /SwitchMatrix/Row3 -> /SwitchMatrix/Col0
- D31 pad 1: /SwitchMatrix/Row3 -> /SwitchMatrix/Col1
- D32 pad 1: /SwitchMatrix/Row3 -> /SwitchMatrix/Col2
- D33 pad 1: /SwitchMatrix/Row3 -> /SwitchMatrix/Col3
- D34 pad 1: /SwitchMatrix/Row3 -> /SwitchMatrix/Col4
- D35 pad 1: /SwitchMatrix/Row3 -> /SwitchMatrix/Col5
- D36 pad 1: /SwitchMatrix/Row3 -> /SwitchMatrix/Col6
- D37 pad 1: /SwitchMatrix/Row3 -> /SwitchMatrix/Col7
- D42 pad 1: /SwitchMatrix/Row4 -> /SwitchMatrix/Col5
- D43 pad 1: /SwitchMatrix/Row4 -> /SwitchMatrix/Col4
- D44 pad 1: /SwitchMatrix/Row4 -> /SwitchMatrix/Col3
- D45 pad 1: /SwitchMatrix/Row4 -> /SwitchMatrix/Col2
- D46 pad 1: /SwitchMatrix/Row4 -> /SwitchMatrix/Col1
- D47 pad 1: /SwitchMatrix/Row4 -> /SwitchMatrix/Col0
- D500 pad 1: /SwitchMatrix/Row0 -> /SwitchMatrix/Col7
- D501 pad 1: /SwitchMatrix/Row1 -> /SwitchMatrix/Col6
- D502 pad 1: /SwitchMatrix/Row2 -> /SwitchMatrix/Col5
- D503 pad 1: /SwitchMatrix/Row3 -> /SwitchMatrix/Col4
- D504 pad 1: /SwitchMatrix/Row4 -> /SwitchMatrix/Col0
- D505 pad 1: /SwitchMatrix/Row5 -> /SwitchMatrix/Col1
- D506 pad 1: /SwitchMatrix/Row6 -> /SwitchMatrix/Col2
- D507 pad 1: /SwitchMatrix/Row7 -> /SwitchMatrix/Col3
- D52 pad 1: /SwitchMatrix/Row5 -> /SwitchMatrix/Col5
- D53 pad 1: /SwitchMatrix/Row5 -> /SwitchMatrix/Col4
- D54 pad 1: /SwitchMatrix/Row5 -> /SwitchMatrix/Col3
- D55 pad 1: /SwitchMatrix/Row5 -> /SwitchMatrix/Col2
- D56 pad 1: /SwitchMatrix/Row5 -> /SwitchMatrix/Col1
- D57 pad 1: /SwitchMatrix/Row5 -> /SwitchMatrix/Col0
- D60 pad 1: /SwitchMatrix/Row6 -> /SwitchMatrix/Col7
- D61 pad 1: /SwitchMatrix/Row6 -> /SwitchMatrix/Col6
- D62 pad 1: /SwitchMatrix/Row6 -> /SwitchMatrix/Col5
- D63 pad 1: /SwitchMatrix/Row6 -> /SwitchMatrix/Col4
- D64 pad 1: /SwitchMatrix/Row6 -> /SwitchMatrix/Col3
- D65 pad 1: /SwitchMatrix/Row6 -> /SwitchMatrix/Col2
- D66 pad 1: /SwitchMatrix/Row6 -> /SwitchMatrix/Col1
- D67 pad 1: /SwitchMatrix/Row6 -> /SwitchMatrix/Col0
- D70 pad 1: /SwitchMatrix/Row7 -> /SwitchMatrix/Col7
- D71 pad 1: /SwitchMatrix/Row7 -> /SwitchMatrix/Col6
- D72 pad 1: /SwitchMatrix/Row7 -> /SwitchMatrix/Col5
- D73 pad 1: /SwitchMatrix/Row7 -> /SwitchMatrix/Col4
- D74 pad 1: /SwitchMatrix/Row7 -> /SwitchMatrix/Col3
- D75 pad 1: /SwitchMatrix/Row7 -> /SwitchMatrix/Col2
- D76 pad 1: /SwitchMatrix/Row7 -> /SwitchMatrix/Col1
- D77 pad 1: /SwitchMatrix/Row7 -> /SwitchMatrix/Col0
- K10 pad 1: /SwitchMatrix/Col7 -> /SwitchMatrix/Row1
- K11 pad 1: /SwitchMatrix/Col6 -> /SwitchMatrix/Row1
- K12 pad 1: /SwitchMatrix/Col5 -> /SwitchMatrix/Row1
- K13 pad 1: /SwitchMatrix/Col4 -> /SwitchMatrix/Row1
- K14 pad 1: /SwitchMatrix/Col3 -> /SwitchMatrix/Row1
- K15 pad 1: /SwitchMatrix/Col2 -> /SwitchMatrix/Row1
- K20 pad 1: /SwitchMatrix/Col7 -> /SwitchMatrix/Row2
- K21 pad 1: /SwitchMatrix/Col6 -> /SwitchMatrix/Row2
- K22 pad 1: /SwitchMatrix/Col5 -> /SwitchMatrix/Row2
- K23 pad 1: /SwitchMatrix/Col4 -> /SwitchMatrix/Row2
- K24 pad 1: /SwitchMatrix/Col3 -> /SwitchMatrix/Row2
- K25 pad 1: /SwitchMatrix/Col2 -> /SwitchMatrix/Row2
- K26 pad 1: /SwitchMatrix/Col1 -> /SwitchMatrix/Row2
- K27 pad 1: /SwitchMatrix/Col0 -> /SwitchMatrix/Row2
- K30 pad 1: /SwitchMatrix/Col7 -> /SwitchMatrix/Row3
- K31 pad 1: /SwitchMatrix/Col6 -> /SwitchMatrix/Row3
- K32 pad 1: /SwitchMatrix/Col5 -> /SwitchMatrix/Row3
- K33 pad 1: /SwitchMatrix/Col4 -> /SwitchMatrix/Row3
- K34 pad 1: /SwitchMatrix/Col3 -> /SwitchMatrix/Row3
- K35 pad 1: /SwitchMatrix/Col2 -> /SwitchMatrix/Row3
- K36 pad 1: /SwitchMatrix/Col1 -> /SwitchMatrix/Row3
- K37 pad 1: /SwitchMatrix/Col0 -> /SwitchMatrix/Row3
- K42 pad 1: /SwitchMatrix/Col2 -> /SwitchMatrix/Row4
- K43 pad 1: /SwitchMatrix/Col3 -> /SwitchMatrix/Row4
- K44 pad 1: /SwitchMatrix/Col4 -> /SwitchMatrix/Row4
- K45 pad 1: /SwitchMatrix/Col5 -> /SwitchMatrix/Row4
- K46 pad 1: /SwitchMatrix/Col6 -> /SwitchMatrix/Row4
- K47 pad 1: /SwitchMatrix/Col7 -> /SwitchMatrix/Row4
- K52 pad 1: /SwitchMatrix/Col2 -> /SwitchMatrix/Row5
- K53 pad 1: /SwitchMatrix/Col3 -> /SwitchMatrix/Row5
- K54 pad 1: /SwitchMatrix/Col4 -> /SwitchMatrix/Row5
- K55 pad 1: /SwitchMatrix/Col5 -> /SwitchMatrix/Row5
- K56 pad 1: /SwitchMatrix/Col6 -> /SwitchMatrix/Row5
- K57 pad 1: /SwitchMatrix/Col7 -> /SwitchMatrix/Row5
- K60 pad 1: /SwitchMatrix/Col0 -> /SwitchMatrix/Row6
- K61 pad 1: /SwitchMatrix/Col1 -> /SwitchMatrix/Row6
- K62 pad 1: /SwitchMatrix/Col2 -> /SwitchMatrix/Row6
- K63 pad 1: /SwitchMatrix/Col3 -> /SwitchMatrix/Row6
- K64 pad 1: /SwitchMatrix/Col4 -> /SwitchMatrix/Row6
- K65 pad 1: /SwitchMatrix/Col5 -> /SwitchMatrix/Row6
- K66 pad 1: /SwitchMatrix/Col6 -> /SwitchMatrix/Row6
- K67 pad 1: /SwitchMatrix/Col7 -> /SwitchMatrix/Row6
- K70 pad 1: /SwitchMatrix/Col0 -> /SwitchMatrix/Row7
- K71 pad 1: /SwitchMatrix/Col1 -> /SwitchMatrix/Row7
- K72 pad 1: /SwitchMatrix/Col2 -> /SwitchMatrix/Row7
- K73 pad 1: /SwitchMatrix/Col3 -> /SwitchMatrix/Row7
- K74 pad 1: /SwitchMatrix/Col4 -> /SwitchMatrix/Row7
- K75 pad 1: /SwitchMatrix/Col5 -> /SwitchMatrix/Row7
- K76 pad 1: /SwitchMatrix/Col6 -> /SwitchMatrix/Row7
- K77 pad 1: /SwitchMatrix/Col7 -> /SwitchMatrix/Row7
- U1 pad 36: ColSelectA -> RowEnable
- U1 pad 37: ColSelectB -> ColSelectC
- U1 pad 38: ColSelectC -> ColSelectB
- U1 pad 40: RowEnable -> ColSelectA
- U2 pad 1: ColSelectA -> RowSelectA
- U2 pad 10: /SwitchMatrix/Col5 -> /SwitchMatrix/Row5
- U2 pad 11: /SwitchMatrix/Col4 -> /SwitchMatrix/Row4
- U2 pad 12: /SwitchMatrix/Col3 -> /SwitchMatrix/Row3
- U2 pad 13: /SwitchMatrix/Col2 -> /SwitchMatrix/Row2
- U2 pad 14: /SwitchMatrix/Col1 -> /SwitchMatrix/Row1
- U2 pad 15: /SwitchMatrix/Col0 -> /SwitchMatrix/Row0
- U2 pad 2: ColSelectB -> RowSelectB
- U2 pad 3: ColSelectC -> RowSelectC
- U2 pad 6: ColEnable -> RowEnable
- U2 pad 7: /SwitchMatrix/Col7 -> /SwitchMatrix/Row7
- U2 pad 9: /SwitchMatrix/Col6 -> /SwitchMatrix/Row6
- U3 pad 1: /SwitchMatrix/Row7 -> /SwitchMatrix/Col3
- U3 pad 10: RowSelectB -> ColSelectB
- U3 pad 11: RowSelectA -> ColSelectA
- U3 pad 12: /SwitchMatrix/Row0 -> /SwitchMatrix/Col7
- U3 pad 13: /SwitchMatrix/Row1 -> /SwitchMatrix/Col6
- U3 pad 14: /SwitchMatrix/Row2 -> /SwitchMatrix/Col5
- U3 pad 15: /SwitchMatrix/Row3 -> /SwitchMatrix/Col4
- U3 pad 2: /SwitchMatrix/Row6 -> /SwitchMatrix/Col2
- U3 pad 3: /SwitchMatrix/Row5 -> /SwitchMatrix/Col1
- U3 pad 4: /SwitchMatrix/Row4 -> /SwitchMatrix/Col0
- U3 pad 7: RowEnable -> ColEnable
- U3 pad 9: RowSelectC -> ColSelectC
Routing:
- net /SwitchMatrix/Col7: track 500.6 -> 10.2 mm, vias 7 -> 0
- net /SwitchMatrix/Col6: track 451.1 -> 8.97 mm, vias 9 -> 0
- net /SwitchMatrix/Col5: track 414.4 -> 7.26 mm, vias 9 -> 0
- net /SwitchMatrix/Col4: track 388.7 -> 5.62 mm, vias 9 -> 0
- net /SwitchMatrix/Col3: track 345.0 -> 6.08 mm, vias 11 -> 0
- net /SwitchMatrix/Col2: track 309.5 -> 7.72 mm, vias 12 -> 0
- net /SwitchMatrix/Col1: track 182.0 -> 9.37 mm
- net Net-(D30-Pad2): track 142.7 -> 0.00 mm
- net /SwitchMatrix/Row4: track 84.5 -> 222.9 mm, vias 0 -> 2
- net Net-(D20-Pad2): track 134.8 -> 0.00 mm
- net /SwitchMatrix/Row5: track 67.6 -> 202.2 mm, vias 1 -> 2
- net Net-(D0-Pad2): track 132.4 -> 0.00 mm
- net Net-(D10-Pad2): track 130.7 -> 0.00 mm
- net /SwitchMatrix/Row6: track 56.9 -> 185.7 mm, vias 1 -> 2
- net Net-(D31-Pad2): track 127.9 -> 0.00 mm
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Other:
- board size 343 x 150.5 mm -> 340.4 x 121.9 mm
- board text added: "Adafruit BLE"
- board text added: "Battery Holder"
- board text added: "CAPS"
- board text added: "NUM"
- board text added: "TRRS"
- board text added: "USB-C"
- board text removed: "C"
- board text removed: "N"
- board text removed: "Wing it! Keyboard Designed by Sam Vasta 2019 rev. H"

Commit message: Moved custom symbols & footprints into git submodules
Parts:
- JP1: footprint SVastaCustomParts:Adafruit BLE SPI -> SVastaCustomParts:Adafruit_BLE_SPI_wire_tht; moved to B.Cu
- K00, K01, K02, K03, K04, K05, K10, K11, K12, K13, K14, K15, K20, K21, K22, K23, K24, K25, K26, K27, K30, K31, K32, K33, K34, K35, K36, K37, K42, K43, K44, K45, K46, K47, K52, K53, K54, K55, K56, K57, K60, K61, K62, K63, K64, K65, K66, K67, K70, K71, K72, K73, K74, K75, K76, K77: footprint keyswitches:Kailh_socket_via_on_pin_one -> SVastaCustomParts:Kailh_socket_via_on_pin_one
- moved R7 28.4 mm to (395.2, 178.6), turned to 180 degrees
- moved R8 22.7 mm to (412.8, 178.1), turned to 0 degrees
- moved JP1 20.5 mm to (383.5, 193.2)
- moved D302 6.54 mm to (389.4, 175.7)
- moved R18 5.85 mm to (384.5, 175.7)
- moved SW1 0.49 mm to (412.2, 183.0)
Routing:
- net VCC: track 217.0 -> 263.2 mm
- net MOSI: track 28.5 -> 53.6 mm, vias 0 -> 1
- net /IRQ: track 26.3 -> 50.8 mm, vias 0 -> 1
- net SS1: track 30.8 -> 55.3 mm, vias 0 -> 1
- net SCK: track 31.1 -> 55.4 mm, vias 0 -> 1
- net MISO: track 28.1 -> 52.3 mm, vias 0 -> 1
- net /RST: track 45.4 -> 69.3 mm, vias 1 -> 2
- net SCL: track 57.2 -> 38.8 mm
- net /SwitchMatrix/Row0: track 204.6 -> 211.1 mm
- net SDA: track 59.7 -> 53.4 mm
- net /SwitchMatrix/Row1: track 188.4 -> 191.9 mm
- net Net-(D302-Pad1): track 5.21 -> 2.82 mm

Commit message: More layout work
Parts:
- removed the D504 at (431.3, 247.8)
- removed the D505 at (431.3, 251.7)
- added D500: D, SVastaCustomParts:D_MiniMELF_Handsoldering_Shorter_Pads, F.Cu at (408.9, 248.8)
- added D501: D, SVastaCustomParts:D_MiniMELF_Handsoldering_Shorter_Pads, F.Cu at (412.8, 248.8)
- D00, D01, D02, D03, D04, D05, D10, D11, D12, D13, D14, D15, D20, D21, D22, D23, D24, D25, D26, D27, D30, D31, D32, D33, D34, D35, D36, D37, D42, D43, D44, D45, D46, D47, D52, D53, D54, D55, D56, D57, D60, D61, D62, D63, D64, D65, D66, D67, D70, D71, D72, D73, D74, D75, D76, D77: footprint Diode_SMD:D_1806_4516Metric_Pad1.57x1.80mm_HandSolder -> SVastaCustomParts:D_MiniMELF_Handsoldering_Shorter_Pads; moved to B.Cu
- D101, D102: footprint Keyboard_Parts:D_axial -> SVastaCustomParts:D_MiniMELF_Handsoldering_Shorter_Pads
- D502: renamed from D506; footprint Diode_SMD:D_0805_2012Metric_Pad1.15x1.40mm_HandSolder -> SVastaCustomParts:D_MiniMELF_Handsoldering_Shorter_Pads
- D503: renamed from D507; footprint Diode_SMD:D_0805_2012Metric_Pad1.15x1.40mm_HandSolder -> SVastaCustomParts:D_MiniMELF_Handsoldering_Shorter_Pads
- D504: renamed from D503; footprint Diode_SMD:D_0805_2012Metric_Pad1.15x1.40mm_HandSolder -> SVastaCustomParts:D_MiniMELF_Handsoldering_Shorter_Pads
- D505: renamed from D502; footprint Diode_SMD:D_0805_2012Metric_Pad1.15x1.40mm_HandSolder -> SVastaCustomParts:D_MiniMELF_Handsoldering_Shorter_Pads
- D506: renamed from D501; footprint Diode_SMD:D_0805_2012Metric_Pad1.15x1.40mm_HandSolder -> SVastaCustomParts:D_MiniMELF_Handsoldering_Shorter_Pads
- D507: renamed from D500; footprint Diode_SMD:D_0805_2012Metric_Pad1.15x1.40mm_HandSolder -> SVastaCustomParts:D_MiniMELF_Handsoldering_Shorter_Pads
- moved D52 73.2 mm to (467.0, 196.0), turned to 102 degrees
- moved D42 70.2 mm to (462.9, 176.9), turned to 102 degrees
- moved D10 64.2 mm to (265.5, 181.5), turned to 348 degrees
- moved D53 62.5 mm to (486.0, 191.9), turned to 102 degrees
- moved D43 58.6 mm to (482.0, 172.9), turned to 102 degrees
- moved D11 56.5 mm to (280.2, 179.4), turned to 78 degrees
- moved D00 56.2 mm to (269.4, 162.0), turned to 348 degrees
- moved D62 55.6 mm to (471.0, 215.1)
- moved D15 55.6 mm to (357.2, 192.2), turned to 78 degrees
- moved D72 52.8 mm to (473.6, 231.5)
- moved D54 50.4 mm to (504.4, 184.4), turned to 102 degrees
- moved D25 50.2 mm to (353.1, 211.3)
- moved D05 49.9 mm to (361.2, 173.2), turned to 78 degrees
- moved D14 49.6 mm to (338.1, 188.2), turned to 78 degrees
- moved D12 48.4 mm to (300.0, 180.1), turned to 78 degrees
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Routing:
- net /SwitchMatrix/Col0: track 11.4 -> 277.5 mm
- net /SwitchMatrix/Col1: track 9.37 -> 193.7 mm
- net /SwitchMatrix/Col2: track 7.72 -> 170.1 mm
- net /SwitchMatrix/Col3: track 6.08 -> 152.8 mm
- net /SwitchMatrix/Col4: track 5.62 -> 128.0 mm
- net /SwitchMatrix/Col5: track 7.26 -> 109.8 mm
- net /SwitchMatrix/Row0: track 211.1 -> 111.2 mm
- net /SwitchMatrix/Row1: track 191.9 -> 111.0 mm
- net /SwitchMatrix/Col6: track 8.97 -> 50.0 mm
- net /SwitchMatrix/Col7: track 10.2 -> 46.0 mm
- net Net-(D500-Pad2): track 23.4 -> 0.00 mm
- net /SwitchMatrix/Row3: track 172.7 -> 157.1 mm
- net Net-(D10-Pad2): track 0.00 -> 14.6 mm
- net Net-(D20-Pad2): track 0.00 -> 14.2 mm
- net Net-(D00-Pad2): track 0.00 -> 14.1 mm
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Other:
- board text removed: "OFF"
- board text removed: "ON"

Commit message: Minor changes and started trackball module
Parts:
- removed BT1: Battery_Cell, SVastaCustomParts:BatteryHolder_Keystone_1088_1xAA
- removed C1, C2: 22pF, Capacitor_SMD:C_0805_2012Metric_Pad1.15x1.40mm_HandSolder
- removed C10, C11, C12, C9: 1uF, Capacitor_SMD:C_0805_2012Metric_Pad1.15x1.40mm_HandSolder
- removed C13: 10uF, Capacitor_SMD:C_0805_2012Metric_Pad1.15x1.40mm_HandSolder
- removed C3, C4, C5, C6, C8: 0.1uF, Capacitor_SMD:C_0805_2012Metric_Pad1.15x1.40mm_HandSolder
- removed C7: 4.7uF, Capacitor_SMD:C_0805_2012Metric_Pad1.15x1.40mm_HandSolder
- removed D101, D102, D42, D43, D44, D45, D46, D47, D500, D501, D502, D503, D504, D505, D506, D507, D52, D53, D54, D55, D56, D57, D60, D61, D62, D63, D64, D65, D66, D67, D70, D71, D72, D73, D74, D75, D76, D77: D, SVastaCustomParts:D_MiniMELF_Handsoldering_Shorter_Pads
- removed D201: Power Good, LED_SMD:LED_0805_2012Metric_Pad1.15x1.40mm_HandSolder
- removed D202: Charge Complete, LED_SMD:LED_0805_2012Metric_Pad1.15x1.40mm_HandSolder
- removed D203: Charging, LED_SMD:LED_0805_2012Metric_Pad1.15x1.40mm_HandSolder
- removed D301: Power, LED_SMD:LED_0805_2012Metric_Pad1.15x1.40mm_HandSolder
- removed D302: Bat Low, LED_SMD:LED_0805_2012Metric_Pad1.15x1.40mm_HandSolder
- removed K42, K43, K44, K45, K46, K47, K52, K53, K54, K55, K56, K57, K60, K61, K62, K63, K64, K65, K66, K67, K70, K71, K72, K73, K74, K75, K76, K77: KEYSW, SVastaCustomParts:Kailh_socket_via_on_pin_one
- removed L1: 10uH, Inductor_SMD:L_0805_2012Metric_Pad1.15x1.40mm_HandSolder
- removed Q1: PZT3906, Package_TO_SOT_SMD:SOT-223
- removed R1, R10, R17, R2: 10K, Resistor_SMD:R_0805_2012Metric_Pad1.15x1.40mm_HandSolder
- removed R11, R12, R13, R16, R19: 470, Resistor_SMD:R_0805_2012Metric_Pad1.15x1.40mm_HandSolder
- removed R14: 100K, Resistor_SMD:R_0805_2012Metric_Pad1.15x1.40mm_HandSolder
- removed R15: 45K, Resistor_SMD:R_0805_2012Metric_Pad1.15x1.40mm_HandSolder
- removed R18: 220, Resistor_SMD:R_0805_2012Metric_Pad1.15x1.40mm_HandSolder
- removed R20: 10k, Resistor_THT:R_Axial_DIN0204_L3.6mm_D1.6mm_P5.08mm_Horizontal
- removed R3, R4: 5.1K, Resistor_SMD:R_0805_2012Metric_Pad1.15x1.40mm_HandSolder
- removed R5, R6: 22, Resistor_SMD:R_0805_2012Metric_Pad1.15x1.40mm_HandSolder
- removed R7, R8: 4.7K, Resistor_SMD:R_0805_2012Metric_Pad1.15x1.40mm_HandSolder
- removed R9: 1K, Resistor_SMD:R_0805_2012Metric_Pad1.15x1.40mm_HandSolder
- removed SW2: SW_SPDT, SVastaCustomParts:400BWMSP1R2BLKSM6QE‎_rocker_switch
- removed U4: MCP73833, SVastaCustomParts:MCP73833T-AMI-UN
- removed U5: LM8364-2.2, Package_TO_SOT_SMD:SOT-23-5_HandSoldering
- removed U6: LTC3525-5, Package_TO_SOT_SMD:SOT-363_SC-70-6_Handsoldering
- added C101: 1uF, Capacitor_SMD:C_0805_2012Metric_Pad1.15x1.40mm_HandSolder, B.Cu at (228.0, 49.4)
- added C102: 102, Capacitor_SMD:C_0805_2012Metric_Pad1.15x1.40mm_HandSolder, B.Cu at (237.7, 40.5)
- added C103: 0.1uF, Capacitor_SMD:C_0805_2012Metric_Pad1.15x1.40mm_HandSolder, B.Cu at (220.2, 33.5)
- added C104: 0.1uF, Capacitor_SMD:C_0805_2012Metric_Pad1.15x1.40mm_HandSolder, B.Cu at (236.9, 35.8)
- added C105: 0.1uF, Capacitor_SMD:C_0805_2012Metric_Pad1.15x1.40mm_HandSolder, F.Cu at (225.4, 40.1)
- added C106: 0.1uF, Capacitor_SMD:C_0805_2012Metric_Pad1.15x1.40mm_HandSolder, F.Cu at (225.2, 42.4)
- added C107: 4.7uF, Capacitor_SMD:C_0805_2012Metric_Pad1.15x1.40mm_HandSolder, B.Cu at (237.7, 42.8)
- added C108: 22pF, Capacitor_SMD:C_0805_2012Metric_Pad1.15x1.40mm_HandSolder, F.Cu at (218.6, 42.0)
- added C109: 22pF, Capacitor_SMD:C_0805_2012Metric_Pad1.15x1.40mm_HandSolder, F.Cu at (218.6, 37.4)
- added C201: 10nF, Capacitor_SMD:C_0805_2012Metric_Pad1.15x1.40mm_HandSolder, F.Cu at (317.4, 76.9)
- added D403: CONN, LED_SMD:LED_0805_2012Metric_Pad1.15x1.40mm_HandSolder, F.Cu at (344.7, 86.6)
- added J2: TRRS_SJ1-42514, SVastaCustomParts:3.5mm_Cut_out, F.Cu at (351.2, 93.8)
- added JP0: SolderJumper_3_Open, Jumper:SolderJumper-3_P1.3mm_Open_RoundedPad1.0x1.5mm, B.Cu at (324.9, 85.4)
- added JP2: SolderJumper_3_Open, Jumper:SolderJumper-3_P1.3mm_Open_RoundedPad1.0x1.5mm, B.Cu at (330.2, 86.9)
- added OLED1: Conn_01x04, Connector_PinHeader_2.54mm:PinHeader_1x04_P2.54mm_Vertical, F.Cu at (199.5, 42.4)
- added R101: 5.1K, Resistor_SMD:R_0805_2012Metric_Pad1.15x1.40mm_HandSolder, F.Cu at (249.4, 37.8)
- added R102: 5.1K, Resistor_SMD:R_0805_2012Metric_Pad1.15x1.40mm_HandSolder, F.Cu at (249.4, 34.3)
- added R103: 10K, Resistor_SMD:R_0805_2012Metric_Pad1.15x1.40mm_HandSolder, B.Cu at (271.0, 40.1)
- added R104: 22, Resistor_SMD:R_0805_2012Metric_Pad1.15x1.40mm_HandSolder, B.Cu at (239.3, 35.8)
- added R105: 22, Resistor_SMD:R_0805_2012Metric_Pad1.15x1.40mm_HandSolder, B.Cu at (241.6, 35.8)
- added R106: 4.7K, Resistor_SMD:R_0805_2012Metric_Pad1.15x1.40mm_HandSolder, B.Cu at (214.8, 33.3)
- added R107: 4.7K, Resistor_SMD:R_0805_2012Metric_Pad1.15x1.40mm_HandSolder, B.Cu at (214.3, 45.0)
- added R108: 10K, Resistor_SMD:R_0805_2012Metric_Pad1.15x1.40mm_HandSolder, F.Cu at (231.2, 37.4)
- added R201: 10K, Resistor_SMD:R_0805_2012Metric_Pad1.15x1.40mm_HandSolder, B.Cu at (322.0, 81.2)
- added R202: 10K, Resistor_SMD:R_0805_2012Metric_Pad1.15x1.40mm_HandSolder, B.Cu at (321.4, 83.5)
- added R203: 10K, Resistor_SMD:R_0805_2012Metric_Pad1.15x1.40mm_HandSolder, B.Cu at (320.8, 85.7)
- added R204: 10K, Resistor_SMD:R_0805_2012Metric_Pad1.15x1.40mm_HandSolder, B.Cu at (320.2, 88.0)
- added R301: 10K, Resistor_SMD:R_0805_2012Metric_Pad1.15x1.40mm_HandSolder, B.Cu at (334.4, 86.8)
- added R302: 10K, Resistor_SMD:R_0805_2012Metric_Pad1.15x1.40mm_HandSolder, B.Cu at (333.7, 89.2)
- added R401: 470, Resistor_SMD:R_0805_2012Metric_Pad1.15x1.40mm_HandSolder, F.Cu at (255.9, 36.1)
- added R402: 470, Resistor_SMD:R_0805_2012Metric_Pad1.15x1.40mm_HandSolder, F.Cu at (267.5, 36.1)
- added R403: 470, Resistor_SMD:R_0805_2012Metric_Pad1.15x1.40mm_HandSolder, B.Cu at (344.7, 86.6)
- added SPI1: Conn_01x04, Connector_PinHeader_2.54mm:PinHeader_1x04_P2.54mm_Vertical, F.Cu at (265.4, 42.0)
- D00, D01, D02, D03, D04, D05, D10, D11, D12, D13, D14, D15, D20, D21, D22, D23, D24, D25, D26, D27, D30, D31, D32, D33, D34, D35, D36, D37: footprint SVastaCustomParts:D_MiniMELF_Handsoldering_Shorter_Pads -> SVastaCustomParts:D_MiniMELF_Handsoldering_Shorter_Pads_DoubleSided; moved to F.Cu
- D401, D402, X1: moved to B.Cu
- J1: moved to F.Cu
- JP1: value HEADER-1X9 -> SolderJumper_3_Open; footprint SVastaCustomParts:Adafruit_BLE_SPI_wire_tht -> Jumper:SolderJumper-3_P1.3mm_Open_RoundedPad1.0x1.5mm
- K00, K01, K02, K03, K04, K05, K10, K11, K12, K13, K14, K15, K20, K21, K22, K23, K24, K25, K26, K27, K30, K31, K32, K33, K34, K35, K36, K37: footprint SVastaCustomParts:Kailh_socket_via_on_pin_one -> SVastaCustomParts:Kailh_socket_reversible
- U1: footprint Keebio:ATMEGA32U4-AU -> SVastaCustomParts:ATMEGA32U4-AU_FixedMask; moved to B.Cu
- U2: value SN74HC138D‎ -> PI6ULS5V9511AWEX_I2C_HotSwap; footprint SVastaCustomParts:SN74HC_package_d_soic -> SVastaCustomParts:PI6ULS5V9511A_I2C_HotSwap
- U3: value SN74HC251 -> MCP23017_SO; footprint SVastaCustomParts:SN74HC_package_d_soic -> Package_SO:SOIC-28W_7.5x17.9mm_P1.27mm
- moved U1 254.4 mm to (227.2, 39.3), turned to 90 degrees
- moved X1 250.1 mm to (215.5, 39.3), turned to 135 degrees
- moved J1 235.2 mm to (207.3, 39.9)
- moved D401 226.1 mm to (255.9, 36.1), turned to 90 degrees
- moved D402 221.9 mm to (267.5, 36.1), turned to 90 degrees
- moved SW1 214.2 mm to (258.4, 33.9)
- moved USB1 213.6 mm to (246.7, 41.3)
- moved U3 186.0 mm to (332.5, 87.5), turned to 255 degrees
- moved U2 184.6 mm to (320.3, 84.6), turned to 165 degrees
- moved D26 173.6 mm to (322.3, 109.0), turned to 165 degrees
- moved D36 172.2 mm to (318.8, 123.2), turned to 165 degrees
- moved D27 164.8 mm to (341.1, 114.1), turned to 345 degrees
- moved D37 163.4 mm to (337.4, 128.0), turned to 165 degrees
- moved K27 138.9 mm to (346.9, 105.8), turned to 165 degrees
- moved K05 137.4 mm to (303.2, 51.4), turned to 180 degrees
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Connections:
- D402 pad 1: Net-(D401-Pad1) -> Net-(D402-Pad1)
- JP1 pad 1: SCK -> Net-(JP0-Pad1)
- JP1 pad 2: MISO -> Net-(JP1-Pad2)
- JP1 pad 3: MOSI -> Net-(JP0-Pad3)
- K00 pad 1: /SwitchMatrix/Row0 -> Net-(D00-Pad2)
- K00 pad 2: Net-(D00-Pad2) -> /SwitchMatrix/Row0
- K01 pad 1: /SwitchMatrix/Row0 -> Net-(D01-Pad2)
- K01 pad 2: Net-(D01-Pad2) -> /SwitchMatrix/Row0
- K02 pad 1: /SwitchMatrix/Row0 -> Net-(D02-Pad2)
- K02 pad 2: Net-(D02-Pad2) -> /SwitchMatrix/Row0
- K03 pad 1: /SwitchMatrix/Row0 -> Net-(D03-Pad2)
- K03 pad 2: Net-(D03-Pad2) -> /SwitchMatrix/Row0
- K04 pad 1: /SwitchMatrix/Row0 -> Net-(D04-Pad2)
- K04 pad 2: Net-(D04-Pad2) -> /SwitchMatrix/Row0
- K05 pad 1: /SwitchMatrix/Row0 -> Net-(D05-Pad2)
- K05 pad 2: Net-(D05-Pad2) -> /SwitchMatrix/Row0
- K26 pad 1: /SwitchMatrix/Row2 -> Net-(D26-Pad2)
- K26 pad 2: Net-(D26-Pad2) -> /SwitchMatrix/Row2
- K27 pad 1: /SwitchMatrix/Row2 -> Net-(D27-Pad2)
- K27 pad 2: Net-(D27-Pad2) -> /SwitchMatrix/Row2
- U1 pad 10: MOSI -> /MOSI
- U1 pad 11: MISO -> /MISO
- U1 pad 12: /IRQ -> Net-(U1-Pad12)
- U1 pad 27: /CapsLock -> Net-(U1-Pad27)
- U1 pad 28: /NumLock -> Net-(U1-Pad28)
- U1 pad 29: RowSelectA -> Net-(U1-Pad29)
- U1 pad 30: /VbatMonitor -> Net-(U1-Pad30)
- U1 pad 31: RowSelectB -> Net-(U1-Pad31)
- U1 pad 32: RowSelectC -> Net-(U1-Pad32)
- U1 pad 36: RowEnable -> /NumLock
- U1 pad 37: ColSelectC -> /CapsLock
- U1 pad 38: ColSelectB -> Net-(U1-Pad38)
- U1 pad 39: ColEnable -> Net-(U1-Pad39)
- U1 pad 40: ColSelectA -> Net-(U1-Pad40)
- U1 pad 41: ColValue -> Net-(U1-Pad41)
- U1 pad 8: SS1 -> /SS
- U1 pad 9: SCK -> /SCK
- U2 pad 1: RowSelectA -> Net-(C201-Pad1)
- U2 pad 2: RowSelectB -> SCL_Clean
- U2 pad 3: RowSelectC -> SCL
- U2 pad 5: GND -> Net-(R204-Pad1)
- U2 pad 6: RowEnable -> SDA
- U2 pad 7: /SwitchMatrix/Row7 -> SDA_Clean
- U2 pad 8: GND -> VCC
- U3 pad 1: /SwitchMatrix/Col3 -> /SwitchMatrix/Col0
- U3 pad 10: ColSelectB -> GND
- U3 pad 11: ColSelectA -> Net-(U3-Pad11)
- U3 pad 12: /SwitchMatrix/Col7 -> SCL_Clean
- U3 pad 13: /SwitchMatrix/Col6 -> SDA_Clean
- U3 pad 14: /SwitchMatrix/Col5 -> Net-(U3-Pad14)
- U3 pad 15: /SwitchMatrix/Col4 -> Net-(JP0-Pad2)
- U3 pad 16: VCC -> Net-(JP1-Pad2)
- U3 pad 2: /SwitchMatrix/Col2 -> /SwitchMatrix/Col1
- U3 pad 3: /SwitchMatrix/Col1 -> /SwitchMatrix/Col2
- U3 pad 4: /SwitchMatrix/Col0 -> /SwitchMatrix/Col3
- U3 pad 5: ColValue -> /SwitchMatrix/Col4
- U3 pad 6: Net-(U3-Pad6) -> /IO_Connected
- U3 pad 7: ColEnable -> Net-(U3-Pad7)
- U3 pad 8: GND -> Net-(U3-Pad8)
- U3 pad 9: ColSelectC -> VCC
- USB1 pad A4: /BMS/USB_V+ -> VCC
- USB1 pad A9: /BMS/USB_V+ -> VCC
- USB1 pad B4: /BMS/USB_V+ -> VCC
- USB1 pad B9: /BMS/USB_V+ -> VCC
Routing:
- net /SwitchMatrix/Row4: track 219.1 -> 0.00 mm, vias 2 -> 0
- net /SwitchMatrix/Row5: track 199.1 -> 0.00 mm, vias 2 -> 0
- net /SwitchMatrix/Row6: track 191.3 -> 0.00 mm, vias 2 -> 0
- net SCL: track 38.8 -> 227.4 mm, vias 0 -> 4
- net /SwitchMatrix/Row7: track 188.3 -> 0.00 mm, vias 2 -> 0
- net SDA: track 53.4 -> 241.3 mm, vias 0 -> 4
- net /RST: track 69.3 -> 171.9 mm, vias 2 -> 3
- net /BMS/USB_V+: track 101.5 -> 0.00 mm
- net /SwitchMatrix/Row0: track 111.2 -> 191.2 mm, vias 2 -> 0
- net /VbatMonitor: track 72.7 -> 0.00 mm, vias 2 -> 0
- net /SwitchMatrix/Row1: track 111.0 -> 173.6 mm, vias 2 -> 0
- net /SwitchMatrix/Row3: track 157.1 -> 216.0 mm
- net Net-(R12-Pad2): track 56.6 -> 0.00 mm, vias 2 -> 0
- net SCK: track 55.4 -> 0.00 mm, vias 1 -> 0
- net SS1: track 55.3 -> 0.00 mm, vias 1 -> 0
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- added copper zone on F.Cu, net GND
- removed copper zone on B.Cu, net GND
Other:
- board size 340.4 x 121.9 mm -> 164 x 102.9 mm
- board text added: "5V"
- board text added: "C"
- board text added: "GND"
- board text added: "MI"
- board text added: "MO"
- board text added: "N"
- board text added: "SCK"
- board text added: "SCL"
- board text added: "SDA"
- board text added: "SS"
- board text removed: "Adafruit BLE"
- board text removed: "Bat Low"
- board text removed: "Bat On"
- board text removed: "Battery Holder"
- board text removed: "CAPS"
- board text removed: "Charging"
- board text removed: "Done"
- board text removed: "NUM"
- board text removed: "TRRS"
- board text removed: "USB"
- board text removed: "USB-C"
