File: pcb/Keeb.kicad_pcb (KiCad board)
At the start: 2 copper layers, 145.5 x 73.3 mm, 99 parts, among them J2 TRRS_SJ1-42514, K00 KEYSW, K01 KEYSW, K02 KEYSW, K03 KEYSW, K04 KEYSW, K05 KEYSW, K10 KEYSW, K11 KEYSW, K12 KEYSW, K13 KEYSW, K14 KEYSW, K15 KEYSW, K20 KEYSW, K21 KEYSW, K22 KEYSW, K23 KEYSW, K24 KEYSW, K25 KEYSW, K26 KEYSW, K30 KEYSW, K31 KEYSW, K32 KEYSW, K33 KEYSW, K34 KEYSW, K35 KEYSW, K36 KEYSW, SW1 SW_RST, U1 ATMEGA32U4, U2 PI6ULS5V9511AWEX_I2C_HotSwap, U3 MCP23017_SO, X1 XTAL_GND

Commit message: Finished new layout
Parts:
- removed D401 (x2): CAPS, LED_SMD:LED_0805_2012Metric_Pad1.15x1.40mm_HandSolder
- removed D402 (x2): NUM, LED_SMD:LED_0805_2012Metric_Pad1.15x1.40mm_HandSolder
- removed D403 (x2): CONN, LED_SMD:LED_0805_2012Metric_Pad1.15x1.40mm_HandSolder
- removed the OLED1 at (323.9, 59.6)
- removed the OLED1 at (323.9, 93.8)
- removed R401, R402, R403: 470, Resistor_SMD:R_0805_2012Metric_Pad1.15x1.40mm_HandSolder
- added OLED1: Conn_01x04, SVastaCustomParts:128x64px_OLED_I2C, F.Cu at (329.8, 72.2)
- added OLED1: Conn_01x04, SVastaCustomParts:128x64px_OLED_I2C, B.Cu at (329.8, 72.2)
- R103, R107: moved to B.Cu
- R106: moved to F.Cu
- U3: footprint Package_SO:SOIC-28W_7.5x17.9mm_P1.27mm -> SVastaCustomParts:MCP231017-SOIC28-wide
- moved R103 43.5 mm to (324.4, 101.6)
- moved R202 20.4 mm to (314.7, 82.6), turned to 0 degrees
- moved 1 17.2 mm to (322.5, 87.4)
- moved R301 17.2 mm to (324.4, 97.2)
- moved R302 17.2 mm to (320.5, 97.2)
- moved 2 17.2 mm to (322.5, 90.3)
- moved 4 17.2 mm to (322.5, 93.3)
- moved U3 17.2 mm to (322.5, 95.2)
- moved R201 16.4 mm to (314.7, 79.6), turned to 0 degrees
- moved C201 12.4 mm to (314.7, 76.7), turned to 0 degrees
- moved U2 12.4 mm to (314.7, 76.7), turned to 0 degrees
- moved R204 8.66 mm to (314.7, 73.8), turned to 180 degrees
- moved R106 6.63 mm to (323.4, 57.7), turned to 180 degrees
- moved R107 6.63 mm to (323.4, 57.7), turned to 180 degrees
- moved C104 5.54 mm to (325.4, 82.0)
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Connections:
- U3 pad 28: /IO_Connected -> Net-(U3-Pad28)
Routing:
- net SDA: track 105.9 -> 66.1 mm, vias 5 -> 3
- net /NumLock: track 32.3 -> 0.00 mm, vias 2 -> 0
- net /CapsLock: track 28.5 -> 0.00 mm, vias 1 -> 0
- net GND: track 79.9 -> 55.7 mm, vias 42 -> 34
- net /IO_Connected: track 22.3 -> 0.00 mm, vias 2 -> 0
- net /SwitchMatrix/Row0: track 138.7 -> 157.9 mm
- net SCL_Clean: track 11.0 -> 26.0 mm
- net /SwitchMatrix/Col4: track 127.7 -> 113.1 mm
- net /SwitchMatrix/Col0: track 206.2 -> 191.7 mm
- net /SwitchMatrix/Col1: track 184.7 -> 170.3 mm
- net /SwitchMatrix/Col2: track 166.8 -> 152.4 mm
- net /SwitchMatrix/Col3: track 148.9 -> 134.5 mm
- net SDA_Clean: track 15.5 -> 28.1 mm
- net /SwitchMatrix/Row1: track 130.7 -> 142.8 mm
- net /SwitchMatrix/Row3: track 147.1 -> 136.7 mm
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Other:
- board text removed: "C"
- board text removed: "N"
