File: pcb/Keeb.sch (KiCad schematic (older format))
At the start: 43 parts, among them J1 TRRS_SJ1-42514, J2 TRRS_SJ1-42514, SW1 SW_RST, U1 ATMEGA32U4, U2 PI6ULS5V9511AWEX_I2C_HotSwap, U3 MCP23017_SO, X1 XTAL_GND

Commit message: Fixed layout to support trackball over SPI
Parts:
- SPI1: footprint Connector_PinHeader_2.54mm:PinHeader_1x04_P2.54mm_Vertical -> Connector_PinHeader_2.54mm:PinHeader_2x04_P2.54mm_Vertical; symbol Connector_Generic:Conn_01x04 -> Connector_Generic:Conn_01x08
Connections:
- net GND: now also SPI1.8 (Pin_8)
- net RST: now also SPI1.6 (Pin_6)
- net SCL: now also J1.3, J2.3; no longer J1.2, J2.2
- net SDA: now also J1.4, J2.4; no longer J1.3, J2.3
- net VCC: now also J1.2, J2.2, SPI1.7 (Pin_7); no longer J1.4, J2.4
- net SS2: now reaches U1.12 (PB7/~RTS)
- net SS2: now also SPI1.4 (Pin_4)
- net SS renamed SS1
- net SS1: now also SPI1.5 (Pin_5); no longer SPI1.4 (Pin_4)
Changed lines of the file:
@@
 EESchema Schematic File Version 4
-LIBS:Keeb-cache
 EELAYER 30 0
 EELAYER END
@@
 Wire Wire Line
 	6700 4350 6850 4350
-Text GLabel 9350 1200 0    50   Input ~ 0
+Text GLabel 9350 1100 0    50   Input ~ 0
 SCL
 Text GLabel 3800 4150 0    50   Input ~ 0
@@
 L power:VCC #PWR0129
 U 1 1 5E03963C
-P 9350 1000
-F 0 "#PWR0129" H 9350 850 50  0001 C CNN
-F 1 "VCC" V 9350 1150 50  0000 L CNN
-F 2 "" H 9350 1000 50  0001 C CNN
-F 3 "" H 9350 1000 50  0001 C CNN
-	1    9350 1000
-	0    -1   -1   0
-$EndComp
-Text GLabel 9350 1100 0    50   Input ~ 0
+P 9350 1200
+F 0 "#PWR0129" H 9350 1050 50  0001 C CNN
+F 1 "VCC" V 9350 1350 50  0000 L CNN
+F 2 "" H 9350 1200 50  0001 C CNN
+F 3 "" H 9350 1200 50  0001 C CNN
+	1    9350 1200
+	0    -1   -1   0
+$EndComp
+Text GLabel 9350 1000 0    50   Input ~ 0
 SDA
 Text Label 10150 5950 2    50   ~ 0
@@
 	0    -1   -1   0
 $EndComp
-Text GLabel 9350 1800 0    50   Input ~ 0
+Text GLabel 9350 1700 0    50   Input ~ 0
 SCL
 $Comp
@@
 	-1   0    0    -1
 $EndComp
-$Comp
-L power:VCC #PWR010
-U 1 1 5F1C2196
-P 9350 1600
-F 0 "#PWR010" H 9350 1450 50  0001 C CNN
-F 1 "VCC" V 9350 1750 50  0000 L CNN
-F 2 "" H 9350 1600 50  0001 C CNN
-F 3 "" H 9350 1600 50  0001 C CNN
-	1    9350 1600
-	0    -1   -1   0
-$EndComp
-Text GLabel 9350 1700 0    50   Input ~ 0
+Text GLabel 9350 1600 0    50   Input ~ 0
 SDA
 Wire Wire Line
@@
 Wire Wire Line
 	9350 1700 9800 1700
-Wire Wire Line
-	9350 1800 9800 1800
 Wire Notes Line
 	11050 750  11050 2050
@@
 Wire Wire Line
 	6150 6200 5700 6200
-Text Label 1150 3000 0    50   ~ 0
+Text Label 1100 3500 0    50   ~ 0
 SCK
-Text Label 1150 2900 0    50   ~ 0
-SS
-Text Label 1150 3200 0    50   ~ 0
+Text Label 1100 3300 0    50   ~ 0
+SS1
+Text Label 1100 3700 0    50   ~ 0
 MISO
-Text Label 1150 3100 0    50   ~ 0
+Text Label 1100 3600 0    50   ~ 0
 MOSI
 $Comp
-L Connector_Generic:Conn_01x04 SPI1
+L Connector_Generic:Conn_01x08 SPI1
 U 1 1 5F321C3F
-P 950 3100
-F 0 "SPI1" H 868 2675 50  0000 C CNN
-F 1 "Conn_01x04" H 868 2766 50  0000 C CNN
-F 2 "Connector_PinHeader_2.54mm:PinHeader_1x04_P2.54mm_Vertical" H 950 3100 50  0001 C CNN
-F 3 "~" H 950 3100 50  0001 C CNN
-	1    950  3100
+P 900 3400
+F 0 "SPI1" H 900 2750 50  0000 C CNN
+F 1 "Conn_01x04" H 900 2850 50  0000 C CNN
+F 2 "Connector_PinHeader_2.54mm:PinHeader_2x04_P2.54mm_Vertical" H 900 3400 50  0001 C CNN
+F 3 "~" H 900 3400 50  0001 C CNN
+	1    900  3400
 	-1   0    0    1
 $EndComp
@@
 SCK
 Text Label 4550 3050 2    50   ~ 0
-SS
+SS1
 Text Label 4550 3350 2    50   ~ 0
 MISO
 Text Label 4550 3250 2    50   ~ 0
 MOSI
+Text Label 4550 3450 2    50   ~ 0
+SS2
+Text Label 1100 3400 0    50   ~ 0
+SS2
+$Comp
+L power:VCC #PWR0122
+U 1 1 5F670E84
+P 1100 3100
+F 0 "#PWR0122" H 1100 2950 50  0001 C CNN
+F 1 "VCC" V 1118 3227 50  0000 L CNN
+F 2 "" H 1100 3100 50  0001 C CNN
+F 3 "" H 1100 3100 50  0001 C CNN
+	1    1100 3100
+	0    1    1    0
+$EndComp
+$Comp
+L power:GND #PWR0132
+U 1 1 5F67C884
+P 1100 3000
+F 0 "#PWR0132" H 1100 2750 50  0001 C CNN
+F 1 "GND" H 1105 2827 50  0000 C CNN
+F 2 "" H 1100 3000 50  0001 C CNN
+F 3 "" H 1100 3000 50  0001 C CNN
+	1    1100 3000
+	0    -1   -1   0
+$EndComp
+Text Label 1100 3200 0    50   ~ 0
+RST
+Wire Wire Line
+	9350 1800 9800 1800
+$Comp
+L power:VCC #PWR010
+U 1 1 5F1C2196
+P 9350 1800
+F 0 "#PWR010" H 9350 1650 50  0001 C CNN
+F 1 "VCC" V 9350 1950 50  0000 L CNN
+F 2 "" H 9350 1800 50  0001 C CNN
+F 3 "" H 9350 1800 50  0001 C CNN
+	1    9350 1800
+	0    -1   -1   0
+$EndComp
 $EndSCHEMATC

Commit message: Fixed issues from test branch
Connections:
- net SwitchMatrix/Col7 is gone; now on net IO_Connected: U3.28 (GPA7)
- net IO_Connected: no longer U3.6 (GPB5)
- net SwitchMatrix/Col5: now also U3.6 (GPB5); no longer U3.26 (GPA5)
- net SwitchMatrix/Col6: now also U3.7 (GPB6); no longer U3.27 (GPA6)
- no-connect marks 3 -> 24
Changed lines of the file:
@@
 	11050 2050 9000 2050
 $Sheet
-S 4950 6150 750  850
+S 4350 6600 750  850
 U 5D9DA1AD
 F0 "SwitchMatrix" 50
 F1 "SwitchMatrix.sch" 50
-F2 "Row0" I L 4950 6200 50
-F3 "Col7" O R 5700 6900 50
-F4 "Row1" I L 4950 6300 50
-F5 "Row2" I L 4950 6400 50
-F6 "Row3" I L 4950 6500 50
-F7 "Col0" O R 5700 6200 50
-F8 "Col1" O R 5700 6300 50
-F9 "Col2" O R 5700 6400 50
-F10 "Col3" O R 5700 6500 50
-F11 "Col4" O R 5700 6600 50
-F12 "Col5" O R 5700 6700 50
-F13 "Col6" O R 5700 6800 50
+F2 "Row0" I L 4350 6650 50
+F3 "Row1" I L 4350 6750 50
+F4 "Row2" I L 4350 6850 50
+F5 "Row3" I L 4350 6950 50
+F6 "Col0" O R 5100 6650 50
+F7 "Col1" O R 5100 6750 50
+F8 "Col2" O R 5100 6850 50
+F9 "Col3" O R 5100 6950 50
+F10 "Col4" O R 5100 7050 50
+F11 "Col5" O R 5100 7150 50
+F12 "Col6" O R 5100 7250 50
 $EndSheet
 $Comp
@@
 Wire Notes Line
 	700  5200 6600 5200
-Wire Wire Line
-	3800 7350 6450 7350
-Wire Wire Line
-	6450 7350 6450 6900
-Wire Wire Line
-	5700 6900 6450 6900
-Wire Wire Line
-	5700 6800 6400 6800
-Wire Wire Line
-	6400 6800 6400 7250
-Wire Wire Line
-	6400 7250 3800 7250
-Wire Wire Line
-	3800 7150 6300 7150
-Wire Wire Line
-	6300 7150 6300 6700
-Wire Wire Line
-	6300 6700 5700 6700
-Wire Wire Line
-	3800 6650 4500 6650
-Wire Wire Line
-	4500 6650 4500 6200
-Wire Wire Line
-	4500 6200 4950 6200
-Wire Wire Line
-	3800 6750 4600 6750
-Wire Wire Line
-	4600 6750 4600 6300
-Wire Wire Line
-	4600 6300 4950 6300
-Wire Wire Line
-	3800 6850 4700 6850
-Wire Wire Line
-	4700 6850 4700 6400
-Wire Wire Line
-	4700 6400 4950 6400
-Wire Wire Line
-	3800 6950 4800 6950
-Wire Wire Line
-	4800 6950 4800 6500
-Wire Wire Line
-	4800 6500 4950 6500
 Wire Wire Line
 	6700 3050 6850 3050
@@
 Wire Wire Line
 	9750 4600 10200 4600
-Text Label 3950 6250 0    50   ~ 0
+Text Label 4150 7700 0    50   ~ 0
 IO_Connected
 Wire Wire Line
-	3800 6250 3950 6250
+	4000 7700 4150 7700
 $Comp
 L Device:LED D?
@@
 Text Notes 7700 3800 0    50   ~ 0
 i2c hot-swap
-Wire Wire Line
-	3800 6150 4400 6150
-Wire Wire Line
-	4400 6150 4400 6000
-Wire Wire Line
-	4400 6000 6400 6000
-Wire Wire Line
-	6400 6000 6400 6600
-Wire Wire Line
-	6400 6600 5700 6600
-Wire Wire Line
-	3800 6050 4350 6050
-Wire Wire Line
-	4350 6050 4350 5950
-Wire Wire Line
-	4350 5950 6350 5950
-Wire Wire Line
-	6350 5950 6350 6500
-Wire Wire Line
-	6350 6500 5700 6500
-Wire Wire Line
-	3800 5950 4300 5950
-Wire Wire Line
-	4300 5950 4300 5850
-Wire Wire Line
-	4300 5850 6300 5850
-Wire Wire Line
-	6300 5850 6300 6400
-Wire Wire Line
-	6300 6400 5700 6400
-Wire Wire Line
-	3800 5850 4250 5850
-Wire Wire Line
-	4250 5850 4250 5800
-Wire Wire Line
-	4250 5800 6200 5800
-Wire Wire Line
-	6200 5800 6200 6300
-Wire Wire Line
-	6200 6300 5700 6300
-Wire Wire Line
-	3800 5750 6150 5750
-Wire Wire Line
-	6150 5750 6150 6200
-Wire Wire Line
-	6150 6200 5700 6200
 Text Label 1100 3500 0    50   ~ 0
 SCK
@@
 	0    -1   -1   0
 $EndComp
+Wire Wire Line
+	5400 6350 5400 7250
+Wire Wire Line
+	5400 7250 5100 7250
+Wire Wire Line
+	5500 6250 5500 7150
+Wire Wire Line
+	5500 7150 5100 7150
+Wire Wire Line
+	5600 6150 5600 7050
+Wire Wire Line
+	5600 7050 5100 7050
+Wire Wire Line
+	5700 6050 5700 6950
+Wire Wire Line
+	5700 6950 5100 6950
+Wire Wire Line
+	5800 5950 5800 6850
+Wire Wire Line
+	5800 6850 5100 6850
+Wire Wire Line
+	5900 5850 5900 6750
+Wire Wire Line
+	5900 6750 5100 6750
+Wire Wire Line
+	3800 6650 4350 6650
+Wire Wire Line
+	4350 6750 3800 6750
+Wire Wire Line
+	3800 6850 4350 6850
+Wire Wire Line
+	4350 6950 3800 6950
+Wire Wire Line
+	5400 6350 3800 6350
+Wire Wire Line
+	3800 6250 5500 6250
+Wire Wire Line
+	5600 6150 3800 6150
+Wire Wire Line
+	3800 6050 5700 6050
+Wire Wire Line
+	5800 5950 3800 5950
+Wire Wire Line
+	3800 5850 5900 5850
+Wire Wire Line
+	3800 5750 6000 5750
+Wire Wire Line
+	6000 5750 6000 6650
+Wire Wire Line
+	6000 6650 5100 6650
+Wire Wire Line
+	3800 7350 4000 7350
+Wire Wire Line
+	4000 7350 4000 7700
+NoConn ~ 3800 6450
+NoConn ~ 3800 7250
+NoConn ~ 3800 7150
+NoConn ~ 3800 7050
+NoConn ~ 2400 6450
+NoConn ~ 2400 6350
+NoConn ~ 6700 2650
+NoConn ~ 6700 2750
+NoConn ~ 6700 2850
+NoConn ~ 6700 2950
+NoConn ~ 4550 4250
+NoConn ~ 4550 4350
+NoConn ~ 4550 4450
+NoConn ~ 6700 4250
+NoConn ~ 6700 4150
+NoConn ~ 6700 4050
+NoConn ~ 6700 3950
+NoConn ~ 6700 3850
+NoConn ~ 6700 3750
+NoConn ~ 6700 3650
+NoConn ~ 6700 3550
 $EndSCHEMATC

Commit message: Finished new layout
Parts:
- removed D401: CAPS, LED_SMD:LED_0805_2012Metric_Pad1.15x1.40mm_HandSolder, symbol Device:LED
- removed D402: NUM, LED_SMD:LED_0805_2012Metric_Pad1.15x1.40mm_HandSolder, symbol Device:LED
- removed D403: CONN, LED_SMD:LED_0805_2012Metric_Pad1.15x1.40mm_HandSolder, symbol Device:LED
- removed J1: TRRS_SJ1-42514, SVastaCustomParts:3.5mm_Cut_out, symbol Keeb-rescue:TRRS_SJ1-42514-SVastaCustomParts-Keeb-rescue
- removed R401, R402, R403: 470, Resistor_SMD:R_0805_2012Metric_Pad1.15x1.40mm_HandSolder, symbol Device:R
- OLED1: footprint Connector_PinHeader_2.54mm:PinHeader_1x04_P2.54mm_Vertical -> SVastaCustomParts:128x64px_OLED_I2C
- U3: footprint Package_SO:SOIC-28W_7.5x17.9mm_P1.27mm -> SVastaCustomParts:MCP231017-SOIC28-wide
Connections:
- net IO_Connected: no longer names the net of U3.28 (GPA7)
- no-connect marks 24 -> 25
Changed lines of the file:
@@
 Wire Wire Line
 	6700 4350 6850 4350
-Text GLabel 9350 1100 0    50   Input ~ 0
-SCL
 Text GLabel 3800 4150 0    50   Input ~ 0
 SDA
@@
 Wire Wire Line
 	3950 4750 3800 4750
-$Comp
-L Keeb-rescue:TRRS_SJ1-42514-SVastaCustomParts-Keeb-rescue J1
-U 1 1 5D8C84D5
-P 10050 750
-F 0 "J1" H 9822 501 50  0000 R CNN
-F 1 "TRRS_SJ1-42514" H 9822 410 50  0000 R CNN
-F 2 "SVastaCustomParts:3.5mm_Cut_out" H 10050 150 50  0000 C CNN
-F 3 "https://www.cui.com/product/resource/sj1-4251x-series.pdf" H 10050 750 50  0001 C CNN
-	1    10050 750
-	-1   0    0    -1
-$EndComp
 Text Notes 1250 5150 2    50   ~ 0
 Switch matrix
@@
 	1    0    0    -1
 $EndComp
-$Comp
-L power:VCC #PWR0129
-U 1 1 5E03963C
-P 9350 1200
-F 0 "#PWR0129" H 9350 1050 50  0001 C CNN
-F 1 "VCC" V 9350 1350 50  0000 L CNN
-F 2 "" H 9350 1200 50  0001 C CNN
-F 3 "" H 9350 1200 50  0001 C CNN
-	1    9350 1200
-	0    -1   -1   0
-$EndComp
-Text GLabel 9350 1000 0    50   Input ~ 0
-SDA
-Text Label 10150 5950 2    50   ~ 0
-CapsLock
-Text Label 10150 6300 2    50   ~ 0
-NumLock
 Wire Notes Line
 	700  5050 700  7750
 Wire Notes Line
 	6600 5200 6600 7750
-$Comp
-L Device:R R?
-U 1 1 5DC64F1A
-P 10600 6300
-AR Path="/5DF457A9/5DC64F1A" Ref="R?"  Part="1"
-AR Path="/5DC64F1A" Ref="R402"  Part="1"
-F 0 "R402" V 10700 6200 50  0000 L CNN
-F 1 "470" V 10600 6200 50  0000 L CNN
-F 2 "Resistor_SMD:R_0805_2012Metric_Pad1.15x1.40mm_HandSolder" V 10530 6300 50  0001 C CNN
-F 3 "~" H 10600 6300 50  0001 C CNN
-	1    10600 6300
-	0    -1   -1   0
-$EndComp
-$Comp
-L Device:LED D?
-U 1 1 5DC64F13
-P 10300 6300
-AR Path="/5DF457A9/5DC64F13" Ref="D?"  Part="1"
-AR Path="/5DC64F13" Ref="D402"  Part="1"
-F 0 "D402" H 10300 6400 50  0000 C CNN
-F 1 "NUM" H 10300 6500 50  0000 C CNN
-F 2 "LED_SMD:LED_0805_2012Metric_Pad1.15x1.40mm_HandSolder" H 10300 6300 50  0001 C CNN
-F 3 "~" H 10300 6300 50  0001 C CNN
-	1    10300 6300
-	-1   0    0    -1
-$EndComp
 Text Label 6850 3050 0    50   ~ 0
 CapsLock
 Text Label 6850 3150 0    50   ~ 0
 NumLock
-Wire Wire Line
-	9350 900  9800 900
-Wire Wire Line
-	9350 1000 9800 1000
-Wire Wire Line
-	9350 1100 9800 1100
-Wire Wire Line
-	9350 1200 9800 1200
 Wire Notes Line
 	11050 2050 9000 2050
@@
 F 0 "U3" H 3100 7831 50  0000 C CNN
 F 1 "MCP23017_SO" H 3100 7740 50  0000 C CNN
-F 2 "Package_SO:SOIC-28W_7.5x17.9mm_P1.27mm" H 3300 5550 50  0001 L CNN
+F 2 "SVastaCustomParts:MCP231017-SOIC28-wide" H 3300 5550 50  0001 L CNN
 F 3 "http://ww1.microchip.com/downloads/en/DeviceDoc/20001952C.pdf" H 3300 5450 50  0001 L CNN
 	1    3100 6550
@@
 Wire Wire Line
 	2400 6650 2150 6650
-Text Label 10150 5600 2    50   ~ 0
-IO_Connected
 $Comp
 L SVastaCustomParts:PI6ULS5V9511AWEX_I2C_HotSwap U2
@@
 Text GLabel 2250 5750 0    50   Input ~ 0
 SDA_Clean
-$Comp
-L Device:LED D?
-U 1 1 5EFC2556
-P 10300 5600
-AR Path="/5DF457A9/5EFC2556" Ref="D?"  Part="1"
-AR Path="/5EFC2556" Ref="D403"  Part="1"
-F 0 "D403" H 10300 5700 50  0000 C CNN
-F 1 "CONN" H 10300 5800 50  0000 C CNN
-F 2 "LED_SMD:LED_0805_2012Metric_Pad1.15x1.40mm_HandSolder" H 10300 5600 50  0001 C CNN
-F 3 "~" H 10300 5600 50  0001 C CNN
-	1    10300 5600
-	-1   0    0    -1
-$EndComp
 Wire Wire Line
 	9750 4600 10200 4600
-Text Label 4150 7700 0    50   ~ 0
-IO_Connected
-Wire Wire Line
-	4000 7700 4150 7700
-$Comp
-L Device:LED D?
-U 1 1 5DC75EFD
-P 10300 5950
-AR Path="/5DF457A9/5DC75EFD" Ref="D?"  Part="1"
-AR Path="/5DC75EFD" Ref="D401"  Part="1"
-F 0 "D401" H 10300 6050 50  0000 C CNN
-F 1 "CAPS" H 10300 6150 50  0000 C CNN
-F 2 "LED_SMD:LED_0805_2012Metric_Pad1.15x1.40mm_HandSolder" H 10300 5950 50  0001 C CNN
-F 3 "~" H 10300 5950 50  0001 C CNN
-	1    10300 5950
-	-1   0    0    -1
-$EndComp
-$Comp
-L Device:R R?
-U 1 1 5F167B0A
-P 10600 5950
-AR Path="/5DF457A9/5F167B0A" Ref="R?"  Part="1"
-AR Path="/5F167B0A" Ref="R401"  Part="1"
-F 0 "R401" V 10700 5850 50  0000 L CNN
-F 1 "470" V 10600 5850 50  0000 L CNN
-F 2 "Resistor_SMD:R_0805_2012Metric_Pad1.15x1.40mm_HandSolder" V 10530 5950 50  0001 C CNN
-F 3 "~" H 10600 5950 50  0001 C CNN
-	1    10600 5950
-	0    -1   -1   0
-$EndComp
-$Comp
-L Device:R R?
-U 1 1 5F1742C1
-P 10600 5600
-AR Path="/5DF457A9/5F1742C1" Ref="R?"  Part="1"
-AR Path="/5F1742C1" Ref="R403"  Part="1"
-F 0 "R403" V 10700 5500 50  0000 L CNN
-F 1 "470" V 10600 5500 50  0000 L CNN
-F 2 "Resistor_SMD:R_0805_2012Metric_Pad1.15x1.40mm_HandSolder" V 10530 5600 50  0001 C CNN
-F 3 "~" H 10600 5600 50  0001 C CNN
-	1    10600 5600
-	0    -1   -1   0
-$EndComp
 Text GLabel 9350 1700 0    50   Input ~ 0
 SCL
@@
 $EndComp
 $Comp
-L power:GND #PWR0113
-U 1 1 5F38EF97
-P 9350 900
-F 0 "#PWR0113" H 9350 650 50  0001 C CNN
-F 1 "GND" H 9355 727 50  0000 C CNN
-F 2 "" H 9350 900 50  0001 C CNN
-F 3 "" H 9350 900 50  0001 C CNN
-	1    9350 900
-	0    1    1    0
-$EndComp
-$Comp
 L power:GND #PWR0114
 U 1 1 5F39B361
@@
 $EndComp
 Connection ~ 8850 4850
-$Comp
-L power:GND #PWR0123
-U 1 1 5F408FED
-P 10750 5600
-F 0 "#PWR0123" H 10750 5350 50  0001 C CNN
-F 1 "GND" H 10755 5427 50  0000 C CNN
-F 2 "" H 10750 5600 50  0001 C CNN
-F 3 "" H 10750 5600 50  0001 C CNN
-	1    10750 5600
-	0    -1   -1   0
-$EndComp
-$Comp
-L power:GND #PWR0124
-U 1 1 5F415395
-P 10750 5950
-F 0 "#PWR0124" H 10750 5700 50  0001 C CNN
-F 1 "GND" H 10755 5777 50  0000 C CNN
-F 2 "" H 10750 5950 50  0001 C CNN
-F 3 "" H 10750 5950 50  0001 C CNN
-	1    10750 5950
-	0    -1   -1   0
-$EndComp
-$Comp
-L power:GND #PWR0125
-U 1 1 5F42168B
-P 10750 6300
-F 0 "#PWR0125" H 10750 6050 50  0001 C CNN
-F 1 "GND" H 10755 6127 50  0000 C CNN
-F 2 "" H 10750 6300 50  0001 C CNN
-F 3 "" H 10750 6300 50  0001 C CNN
-	1    10750 6300
-	0    -1   -1   0
-$EndComp
 Wire Wire Line
 	6700 4450 6900 4450
@@
 F 0 "OLED1" H 8030 5592 50  0000 L CNN
 F 1 "Conn_01x04" H 8030 5501 50  0000 L CNN
-F 2 "Connector_PinHeader_2.54mm:PinHeader_1x04_P2.54mm_Vertical" H 7950 5600 50  0001 C CNN
+F 2 "SVastaCustomParts:128x64px_OLED_I2C" H 7950 5600 50  0001 C CNN
 F 3 "~" H 7950 5600 50  0001 C CNN
 	1    7950 5600
@@
 Wire Wire Line
 	6000 6650 5100 6650
-Wire Wire Line
-	3800 7350 4000 7350
-Wire Wire Line
-	4000 7350 4000 7700
 NoConn ~ 3800 6450
 NoConn ~ 3800 7250
@@
 NoConn ~ 6700 3650
 NoConn ~ 6700 3550
+NoConn ~ 3800 7350
 $EndSCHEMATC
