File: pcb/pcb_main/SwitchMatrix.sch (KiCad schematic (older format))
At the start: 112 parts, among them K00 KEYSW, K01 KEYSW, K02 KEYSW, K03 KEYSW, K04 KEYSW, K05 KEYSW, K10 KEYSW, K11 KEYSW, K12 KEYSW, K13 KEYSW, K14 KEYSW, K15 KEYSW, K20 KEYSW, K21 KEYSW, K22 KEYSW, K23 KEYSW, K24 KEYSW, K25 KEYSW, K26 KEYSW, K27 KEYSW, K30 KEYSW, K31 KEYSW, K32 KEYSW, K33 KEYSW, K34 KEYSW, K35 KEYSW, K36 KEYSW, K37 KEYSW, K42 KEYSW, K43 KEYSW, K44 KEYSW, K45 KEYSW, K46 KEYSW, K47 KEYSW, K52 KEYSW, K53 KEYSW, K54 KEYSW, K55 KEYSW, K56 KEYSW, K57 KEYSW, K60 KEYSW, K61 KEYSW, K62 KEYSW, K63 KEYSW, K64 KEYSW, K65 KEYSW, K66 KEYSW, K67 KEYSW, K70 KEYSW, K71 KEYSW, K72 KEYSW, K73 KEYSW, K74 KEYSW, K75 KEYSW, K76 KEYSW, K77 KEYSW

Commit message: First pass at split pcb design completed
Parts:
- D00, D01, D02, D03, D04, D05, D10, D11, D12, D13, D14, D15, D20, D21, D22, D23, D24, D25, D26, D27, D30, D31, D32, D33, D34, D35, D36, D37, D42, D43, D44, D45, D46, D47, D52, D53, D54, D55, D56, D57, D60, D61, D62, D63, D64, D65, D66, D67, D70, D71, D72, D73, D74, D75, D76, D77: symbol Keyboard_Parts:D -> Keeb-rescue:D-Keyboard_Parts
- K00, K01, K02, K03, K04, K05, K10, K11, K12, K13, K14, K15, K20, K21, K22, K23, K24, K25, K26, K27, K30, K31, K32, K33, K34, K35, K36, K37, K42, K43, K44, K45, K46, K47, K52, K53, K54, K55, K56, K57, K60, K61, K62, K63, K64, K65, K66, K67, K70, K71, K72, K73, K74, K75, K76, K77: symbol Keyboard_Parts:KEYSW -> Keeb-rescue:KEYSW-Keyboard_Parts
