File: pcb/Board/Board.sch (KiCad schematic (older format))
At the start: 14 parts, among them J1 Conn_01x04_Female, J2 TRRS_SJ1-42514, U2 PI6ULS5V9511AWEX_I2C_HotSwap, U3 MCP23017_SO

Commit message: updaaaaaaates
Parts:
- added J3: Conn_01x12_Female, Connector_PinHeader_2.54mm:PinHeader_1x12_P2.54mm_Vertical, symbol Connector:Conn_01x12_Female
- U3: footprint SVastaCustomParts:MCP231017-SOIC28-wide -> Package_SO:SSOP-28_5.3x10.2mm_P0.65mm
Connections:
- net SwitchMatrix/Col0: now also J3.1 (Pin_1)
- net SwitchMatrix/Col1: now also J3.2 (Pin_2)
- net SwitchMatrix/Col2: now also J3.3 (Pin_3)
- net SwitchMatrix/Col3: now also J3.4 (Pin_4)
- net SwitchMatrix/Col4: now also J3.5 (Pin_5)
- net SwitchMatrix/Col5: now also J3.6 (Pin_6)
- net SwitchMatrix/Col6: now also J3.7 (Pin_7)
- net SwitchMatrix/Row0: now also J3.9 (Pin_9)
- net SwitchMatrix/Row1: now also J3.10 (Pin_10)
- net SwitchMatrix/Row2: now also J3.11 (Pin_11)
- net SwitchMatrix/Row3: now also J3.12 (Pin_12)
Changed lines of the file:
@@
 F 0 "U3" H 3050 3431 50  0000 C CNN
 F 1 "MCP23017_SO" H 3050 3340 50  0000 C CNN
-F 2 "SVastaCustomParts:MCP231017-SOIC28-wide" H 3250 1150 50  0001 L CNN
+F 2 "Package_SO:SSOP-28_5.3x10.2mm_P0.65mm" H 3250 1150 50  0001 L CNN
 F 3 "http://ww1.microchip.com/downloads/en/DeviceDoc/20001952C.pdf" H 3250 1050 50  0001 L CNN
 	1    3050 2150
@@
 	5850 2350 5050 2350
 Wire Wire Line
-	3750 2250 4300 2250
-Wire Wire Line
-	4300 2350 3750 2350
-Wire Wire Line
-	3750 2450 4300 2450
-Wire Wire Line
-	4300 2550 3750 2550
+	4300 2550 4000 2550
 Wire Wire Line
 	5350 1950 3750 1950
@@
 	0    -1   -1   0
 $EndComp
+$Comp
+L Connector:Conn_01x12_Female J3
+U 1 1 5FBDE2F6
+P 6500 1850
+F 0 "J3" H 6528 1826 50  0000 L CNN
+F 1 "Conn_01x12_Female" H 6528 1735 50  0000 L CNN
+F 2 "Connector_PinHeader_2.54mm:PinHeader_1x12_P2.54mm_Vertical" H 6500 1850 50  0001 C CNN
+F 3 "~" H 6500 1850 50  0001 C CNN
+	1    6500 1850
+	1    0    0    -1
+$EndComp
+Wire Wire Line
+	5950 1350 6300 1350
+Connection ~ 5950 1350
+Wire Wire Line
+	6300 1450 5850 1450
+Connection ~ 5850 1450
+Wire Wire Line
+	5750 1550 6300 1550
+Connection ~ 5750 1550
+Wire Wire Line
+	6300 1650 5650 1650
+Connection ~ 5650 1650
+Wire Wire Line
+	5550 1750 6300 1750
+Connection ~ 5550 1750
+Wire Wire Line
+	5450 1850 6300 1850
+Connection ~ 5450 1850
+Wire Wire Line
+	5350 1950 6300 1950
+Connection ~ 5350 1950
+Wire Wire Line
+	3750 2450 4050 2450
+Wire Wire Line
+	4300 2350 4100 2350
+Wire Wire Line
+	3750 2250 4150 2250
+Wire Wire Line
+	6300 2150 6150 2150
+Wire Wire Line
+	6150 2150 6150 3150
+Wire Wire Line
+	6150 3150 4150 3150
+Wire Wire Line
+	4150 3150 4150 2250
+Connection ~ 4150 2250
+Wire Wire Line
+	4150 2250 4300 2250
+Wire Wire Line
+	4100 2350 4100 3200
+Wire Wire Line
+	4100 3200 6200 3200
+Wire Wire Line
+	6200 3200 6200 2250
+Wire Wire Line
+	6200 2250 6300 2250
+Connection ~ 4100 2350
+Wire Wire Line
+	4100 2350 3750 2350
+Wire Wire Line
+	6300 2350 6250 2350
+Wire Wire Line
+	6250 2350 6250 3250
+Wire Wire Line
+	6250 3250 4050 3250
+Wire Wire Line
+	4050 3250 4050 2450
+Connection ~ 4050 2450
+Wire Wire Line
+	4050 2450 4300 2450
+Wire Wire Line
+	4000 2550 4000 3300
+Wire Wire Line
+	4000 3300 6300 3300
+Wire Wire Line
+	6300 3300 6300 2450
+Connection ~ 4000 2550
+Wire Wire Line
+	4000 2550 3750 2550
 $EndSCHEMATC

Commit message: Changed i/o expander to ssop package
Parts:
- removed J2: TRRS_SJ1-42514, SVastaCustomParts:3.5mm_Cut_out, symbol Keeb-rescue:TRRS_SJ1-42514-SVastaCustomParts-Keeb-rescue
Connections:
- net RST is gone; now on an unnamed net: U3.18 (~RESET~)
- no-connect marks 7 -> 8
Changed lines of the file:
@@
 Wire Notes Line
 	650  800  6550 800
-Text Label 2100 2250 0    50   ~ 0
-RST
-Wire Wire Line
-	2350 2250 2100 2250
 $Comp
 L SVastaCustomParts:PI6ULS5V9511AWEX_I2C_HotSwap U2
@@
 Wire Wire Line
 	2750 4500 3200 4500
-Text GLabel 1000 6350 0    50   Input ~ 0
-SCL
-$Comp
-L Keeb-rescue:TRRS_SJ1-42514-SVastaCustomParts-Keeb-rescue J2
-U 1 1 5F1C218A
-P 1700 6000
-F 0 "J2" H 1472 5751 50  0000 R CNN
-F 1 "TRRS_SJ1-42514" H 1472 5660 50  0000 R CNN
-F 2 "SVastaCustomParts:3.5mm_Cut_out" H 1700 5400 50  0000 C CNN
-F 3 "https://www.cui.com/product/resource/sj1-4251x-series.pdf" H 1700 6000 50  0001 C CNN
-	1    1700 6000
-	-1   0    0    -1
-$EndComp
-Text GLabel 1000 6250 0    50   Input ~ 0
-SDA
-Wire Wire Line
-	1000 6150 1450 6150
-Wire Wire Line
-	1000 6250 1450 6250
-Wire Wire Line
-	1000 6350 1450 6350
 Wire Notes Line
 	2700 5400 2700 6700
 Wire Notes Line
 	650  6700 650  5250
-$Comp
-L power:GND #PWR0114
-U 1 1 5F39B361
-P 1000 6150
-F 0 "#PWR0114" H 1000 5900 50  0001 C CNN
-F 1 "GND" H 1005 5977 50  0000 C CNN
-F 2 "" H 1000 6150 50  0001 C CNN
-F 3 "" H 1000 6150 50  0001 C CNN
-	1    1000 6150
-	0    1    1    0
-$EndComp
 $Comp
 L power:GND #PWR0121
@@
 i2c hot-swap
 Wire Wire Line
-	1000 6450 1450 6450
-$Comp
-L power:VCC #PWR010
-U 1 1 5F1C2196
-P 1000 6450
-F 0 "#PWR010" H 1000 6300 50  0001 C CNN
-F 1 "VCC" V 1000 6600 50  0000 L CNN
-F 2 "" H 1000 6450 50  0001 C CNN
-F 3 "" H 1000 6450 50  0001 C CNN
-	1    1000 6450
-	0    -1   -1   0
-$EndComp
-Wire Wire Line
 	5350 1950 5350 2850
 Wire Wire Line
@@
 Wire Wire Line
 	4000 2550 3750 2550
+Wire Wire Line
+	2350 2250 2000 2250
+Wire Wire Line
+	2000 2250 2000 1600
+Wire Wire Line
+	2000 1600 1150 1600
+Wire Wire Line
+	1150 1600 1150 2300
+Wire Wire Line
+	1150 2300 1400 2300
+NoConn ~ 6300 2050
 $EndSCHEMATC
