File: pcb/Shield/Shield.sch (KiCad schematic (older format))
At the start: 36 parts, among them J2 TRRS_SJ1-42514, SW1 SW_RST, U1 ATMEGA32U4, U2 PI6ULS5V9511AWEX_I2C_HotSwap, U3 MCP23017_SO, X1 XTAL_GND

Commit message: Split board and shield into separate projects
Parts:
- removed C201: 10nF, Capacitor_SMD:C_0805_2012Metric_Pad1.15x1.40mm_HandSolder, symbol Device:C_Small
- removed JP0, JP1, JP2: SolderJumper_3_Open, Jumper:SolderJumper-3_P1.3mm_Open_RoundedPad1.0x1.5mm, symbol Jumper:SolderJumper_3_Open
- removed OLED1: Conn_01x04, SVastaCustomParts:128x64px_OLED_I2C, symbol Connector_Generic:Conn_01x04
- removed R201, R202, R203, R204, R301, R302: 10K, Resistor_SMD:R_0805_2012Metric_Pad1.15x1.40mm_HandSolder, symbol Device:R
- removed SPI1: Conn_01x04, Connector_PinHeader_2.54mm:PinHeader_2x04_P2.54mm_Vertical, symbol Connector_Generic:Conn_01x08
- removed U2: PI6ULS5V9511AWEX_I2C_HotSwap, SVastaCustomParts:PI6ULS5V9511A_I2C_HotSwap, symbol SVastaCustomParts:PI6ULS5V9511AWEX_I2C_HotSwap
- removed U3: MCP23017_SO, SVastaCustomParts:MCP231017-SOIC28-wide, symbol Interface_Expansion:MCP23017_SO
- added J1, J10, J2, J3, J4, J5, J6, J7, J8, J9: Conn_01x01, Connector_PinHeader_2.54mm:PinHeader_1x01_P2.54mm_Vertical, symbol Connector_Generic:Conn_01x01
- C102: value 102 -> 0.1uF
- J11: renamed from J2; footprint SVastaCustomParts:3.5mm_Cut_out -> Connector_PinHeader_2.54mm:PinHeader_1x02_P2.54mm_Vertical; symbol Keeb-rescue:TRRS_SJ1-42514-SVastaCustomParts-Keeb-rescue -> Connector:Conn_01x02_Female
- SW1: footprint Button_Switch_THT:SW_PUSH_6mm -> SVastaCustomParts:MomentarySwitch_B3U-1000P
Connections:
- net labels removed: CapsLock, NumLock, SCL_Clean, SDA_Clean
- wire segments 174 -> 101
- no-connect marks 25 -> 20
Other:
- note removed: "32x128 i2c OLED"
- note removed: "Switch matrix"
- note removed: "i2c hot-swap"

Commit message: Modified shield to make i2c & usb connections solderless
Parts:
- removed J1, J10, J2, J3, J4, J5, J6, J7, J8, J9: Conn_01x01, Connector_PinHeader_2.54mm:PinHeader_1x01_P2.54mm_Vertical, symbol Connector_Generic:Conn_01x01
- removed J11: TRRS_SJ1-42514, Connector_PinHeader_2.54mm:PinHeader_1x02_P2.54mm_Vertical, symbol Connector:Conn_01x02_Female
- removed R104, R105: 22, Resistor_SMD:R_0805_2012Metric_Pad1.15x1.40mm_HandSolder, symbol Device:R
- removed USB1: USB_C_Receptacle_USB2.0, Connector_USB:USB_C_Receptacle_GCT_USB4085, symbol Connector:USB_C_Receptacle_USB2.0
- added I2C1, I2C2, USB1: Conn_01x04_Female, SVastaCustomParts:Terminal_Block_4pos_On_Shore_Tech., symbol Connector:Conn_01x04_Female
- R101, R102: value 5.1K -> 22R
- renumbered R106 to R104, R107 to R105, R108 to R106
Connections:
- net GND: now also I2C1.1 (Pin_1), I2C2.4 (Pin_4), USB1.1 (Pin_1); no longer R101.1, R102.1
- net SCL: now also I2C1.2 (Pin_2), I2C2.3 (Pin_3)
- net SDA: now also I2C1.3 (Pin_3), I2C2.2 (Pin_2)
- net UsbD+: now also R101.1, U1.4 (D+)
- net UsbD-: now also R102.1, U1.3 (D-)
- net VCC: now also I2C1.4 (Pin_4), I2C2.1 (Pin_1), USB1.4 (Pin_4)
- net at R101.2: now also USB1.3 (Pin_3)
- net at R102.2: now also USB1.2 (Pin_2)
- no-connect marks 20 -> 18
Other:
- note removed: "USB connection advice from:\nhttps://electronics.stackexchange.com/a/373862\nFootprint for digikey part # 2073-USB4085-GF-ACT-ND"
- moved on the sheet: R101, R102
